File: kicad/RCTX.sch (KiCad schematic (older format))
At the start: 25 parts, among them P1 MULTI_PROP_1, P10 USB, P11 BUZZ, P12 SW, P13 LEDS, P14 KEYPAD, P15 MULTI_DIGITAL_1, P16 MULTI_DIGITAL_2, P2 MULTI_PROP_2, P3 SD_CARD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

Commit message: Adding 5110 display
Parts:
- removed C1: C, symbol device:C
- removed P4: LEDs, symbol conn:Conn_01x06
- removed R1: R, symbol device:R
- removed RN1: 15k, Resistors_THT:R_Array_SIP6, symbol device:R_Network05
- added P?: LEDs, symbol conn:Conn_01x04
- added P?: DISPLAY, symbol conn:Conn_01x05
- added RN?: 15k, Resistors_THT:R_Array_SIP6, symbol device:R_Network05
- P8: symbol conn:Conn_01x05 -> conn:Conn_01x04
- RR1: symbol device:R_Network09 -> device:R_Network08
Connections:
- net labels added: +3.3V, +5V, GND
- wire segments 304 -> 311
Other:
- note added: "/CE"
- note added: "/PWM"
- note added: "/RESET"
- note added: "/RF_DETECT"
- note added: "CLK"
- note added: "D/C"
- note added: "DIN"
- note added: "FRQ_METER"
- note added: "PPM_IN"
- note added: "PPM_OUT"
- note removed: "+1.65V"
- note removed: "/LED"
- note removed: "/OE1"
- note removed: "/OE2"
- note removed: "FRQ"
- note removed: "PLL_SYNC"
- note removed: "PPM_IO"
- note removed: "PPM_TX"
- note removed: "SIG"
- moved on the sheet: P1, P11, P12, P13, P14, P15, P16, P2, P5, P6, P9, RR2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

Commit message: Adding footprints
Parts:
- P1, P2: footprint (none) -> Connectors_Samtec:SL-108-X-XX_1x08; symbol conn:Conn_01x08 -> RCTX-rescue:Conn_01x08-conn
- P10: renamed from P9; footprint (none) -> Connectors_Samtec:SL-104-X-XX_1x04; symbol conn:Conn_01x04 -> RCTX-rescue:Conn_01x04-conn
- P11: renamed from P10; footprint (none) -> Connectors_Samtec:SL-105-X-XX_1x05; symbol conn:Conn_01x05 -> RCTX-rescue:Conn_01x05-conn
- P12: renamed from P11; footprint (none) -> Connectors_Samtec:SL-102-X-XX_1x02; symbol conn:Conn_01x02 -> RCTX-rescue:Conn_01x02-conn
- P13: renamed from P12; footprint (none) -> Connectors_Samtec:SL-103-X-XX_1x03; symbol conn:Conn_01x03 -> RCTX-rescue:Conn_01x03-conn
- P14: renamed from P13; footprint (none) -> Connectors_Samtec:SL-104-X-XX_1x04; symbol conn:Conn_01x04 -> RCTX-rescue:Conn_01x04-conn
- P15: renamed from P14; footprint (none) -> Connectors_Samtec:SL-108-X-XX_1x08; symbol conn:Conn_01x08 -> RCTX-rescue:Conn_01x08-conn
- P16: renamed from P15; footprint (none) -> Connectors_Samtec:SL-109-X-XX_1x09; symbol conn:Conn_01x09 -> RCTX-rescue:Conn_01x09-conn
- P17: renamed from P16; footprint (none) -> Connectors_Samtec:SL-109-X-XX_1x09; symbol conn:Conn_01x09 -> RCTX-rescue:Conn_01x09-conn
- P3: footprint (none) -> Connectors_Samtec:SL-104-X-XX_1x04; symbol conn:Conn_01x04 -> RCTX-rescue:Conn_01x04-conn
- P4: renamed from P?; footprint (none) -> Connectors_Samtec:SL-104-X-XX_1x04; symbol conn:Conn_01x04 -> RCTX-rescue:Conn_01x04-conn
- P5: renamed from P?; footprint (none) -> Connectors_Samtec:SL-106-X-XX_1x06; symbol conn:Conn_01x05 -> RCTX-rescue:Conn_01x05-conn
- P6: renamed from P5; footprint (none) -> Connectors_Samtec:SL-108-X-XX_1x08; symbol conn:Conn_01x08 -> RCTX-rescue:Conn_01x08-conn
- P7: renamed from P6; footprint (none) -> Connectors_Samtec:SL-103-X-XX_1x03; symbol conn:Conn_01x03 -> RCTX-rescue:Conn_01x03-conn
- P8: renamed from P7; footprint (none) -> Connectors_Samtec:SL-112-X-XX_1x12; symbol conn:Conn_01x12 -> RCTX-rescue:Conn_01x12-conn
- P9: renamed from P8; footprint (none) -> Connectors_Samtec:SL-104-X-XX_1x04; symbol conn:Conn_01x04 -> RCTX-rescue:Conn_01x04-conn
- RN1: renamed from RN?; symbol device:R_Network05 -> RCTX-rescue:R_Network05-device
- RR1: footprint Resistors_THT:R_Array_SIP10 -> Resistors_THT:R_Array_SIP9; symbol device:R_Network08 -> RCTX-rescue:R_Network08-device
- RR2, RR3: footprint (none) -> Resistors_THT:R_Array_SIP10; symbol device:R_Network09 -> RCTX-rescue:R_Network09-device
- RV1: footprint (none) -> Potentiometers:Potentiometer_Trimmer_ACP_CA6v_Horizontal; symbol device:POT_TRIM -> RCTX-rescue:POT_TRIM-device
- UBW32V1: footprint (none) -> UBW32_v24:UBW32_V24
- ZD1: footprint (none) -> Diodes_THT:D_5W_P5.08mm_Vertical_KathodeUp; symbol device:D_Zener -> RCTX-rescue:D_Zener-device
