File: kicad/RCTX.sch (KiCad schematic (older format))
At the start: 24 parts, among them P1 MULTI_PROP_1, P10 USB, P11 BUZZ, P12 SW, P13 LEDS, P14 KEYPAD, P15 MULTI_DIGITAL_1, P16 MULTI_DIGITAL_2, P2 MULTI_PROP_2, P3 SD_CARD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

Commit message: renaming switches, buttons and trims
Other:
- note added: "ROTARY_01"
- note added: "ROTARY_02"
- note added: "ROTARY_03"
- note added: "ROTARY_04"
- note added: "ROTARY_05"
- note added: "ROTARY_06"
- note added: "ROTARY_07"
- note added: "ROTARY_08"
- note added: "ROTARY_09"
- note added: "ROTARY_10"
- note added: "ROTARY_11"
- note added: "ROTARY_12"
- note removed: "TRIM_1"
- note removed: "TRIM_10"
- note removed: "TRIM_11"
- note removed: "TRIM_12"
- note removed: "TRIM_2"
- note removed: "TRIM_3"
- note removed: "TRIM_4"
- note removed: "TRIM_5"
- note removed: "TRIM_6"
- note removed: "TRIM_7"
- note removed: "TRIM_8"
- note removed: "TRIM_9"
Changed lines of the file:
@@
 Wire Wire Line
 	6150 6350 6150 6450
-$Comp
-L conn:Conn_01x03 P6
-U 1 1 5038EC3A
-P 1750 4750
-F 0 "P6" V 1950 4750 50  0000 C CNN
-F 1 "TX_MOD" V 1850 4750 40  0000 C CNN
-F 2 "" H 1750 4750 60  0001 C CNN
-F 3 "" H 1750 4750 60  0001 C CNN
-	1    1750 4750
-	-1   0    0    -1
-$EndComp
 Text Notes 1450 4700 2    60   ~ 0
 FRQ_METER
@@
 nSRST
 Text Notes 1450 1700 2    60   ~ 0
-TRIM_8
+ROTARY_08
 Text Notes 1450 1600 2    60   ~ 0
-TRIM_7
+ROTARY_07
 Text Notes 1450 1500 2    60   ~ 0
-TRIM_6
+ROTARY_06
 Text Notes 1450 1400 2    60   ~ 0
-TRIM_5
+ROTARY_05
 Text Notes 1450 1300 2    60   ~ 0
-TRIM_4
+ROTARY_04
 Text Notes 1450 1200 2    60   ~ 0
-TRIM_3
+ROTARY_03
 Text Notes 1450 1100 2    60   ~ 0
-TRIM_2
+ROTARY_02
 Text Notes 1450 1000 2    60   ~ 0
-TRIM_1
+ROTARY_01
 Text Notes 1450 1900 2    60   ~ 0
-TRIM_10
+ROTARY_10
 Text Notes 1450 1800 2    60   ~ 0
-TRIM_9
+ROTARY_09
 Text Notes 1450 600  2    60   ~ 0
 H_RIGHT_JOYSTICK
@@
 V_RIGHT_JOYSTICK
 Text Notes 1450 2000 2    60   ~ 0
-TRIM_11
+ROTARY_11
 Text Notes 1450 2100 2    60   ~ 0
-TRIM_12
+ROTARY_12
 Text Notes 1450 800  2    60   ~ 0
 H_LEFT_JOYSTICK
@@
 Wire Wire Line
 	4950 6050 4950 6500
+$Comp
+L conn:Conn_01x03 P6
+U 1 1 5038EC3A
+P 1750 4750
+F 0 "P6" V 1950 4750 50  0000 C CNN
+F 1 "TX_MOD" V 1850 4750 40  0000 C CNN
+F 2 "" H 1750 4750 60  0001 C CNN
+F 3 "" H 1750 4750 60  0001 C CNN
+	1    1750 4750
+	-1   0    0    -1
+$EndComp
 $EndSCHEMATC
