File: kicad/RCTX.sch (KiCad schematic (older format))
At the start: 24 parts, among them P1 MULTI_PROP_1, P10 POWER_IN, P11 USB, P12 BUZZ, P13 SW, P14 LEDS, P15 KEYPAD, P16 MULTI_DIGITAL_1, P17 MULTI_DIGITAL_2, P2 MULTI_PROP_2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

Commit message: Fixing keypad wiring
Connections:
- net +3V3: no longer RR1.1 (common), UBW32V1.86 (3.3V)
- net GND: now also RR1.1 (common), UBW32V1.88 (GND)
Other:
- note added: "ROTARY_01"
- note added: "ROTARY_02"
- note added: "ROTARY_03"
- note added: "ROTARY_04"
- note added: "ROTARY_05"
- note added: "ROTARY_06"
- note added: "ROTARY_07"
- note added: "ROTARY_08"
- note added: "ROTARY_09"
- note added: "ROTARY_10"
- note added: "ROTARY_11"
- note added: "ROTARY_12"
- note removed: "TRIM_1"
- note removed: "TRIM_10"
- note removed: "TRIM_11"
- note removed: "TRIM_12"
- note removed: "TRIM_2"
- note removed: "TRIM_3"
- note removed: "TRIM_4"
- note removed: "TRIM_5"
- note removed: "TRIM_6"
- note removed: "TRIM_7"
- note removed: "TRIM_8"
- note removed: "TRIM_9"
Changed lines of the file:
@@
 nSRST
 Text Notes 1450 1700 2    60   ~ 0
-TRIM_8
+ROTARY_08
 Text Notes 1450 1600 2    60   ~ 0
-TRIM_7
+ROTARY_07
 Text Notes 1450 1500 2    60   ~ 0
-TRIM_6
+ROTARY_06
 Text Notes 1450 1400 2    60   ~ 0
-TRIM_5
+ROTARY_05
 Text Notes 1450 1300 2    60   ~ 0
-TRIM_4
+ROTARY_04
 Text Notes 1450 1200 2    60   ~ 0
-TRIM_3
+ROTARY_03
 Text Notes 1450 1100 2    60   ~ 0
-TRIM_2
+ROTARY_02
 Text Notes 1450 1000 2    60   ~ 0
-TRIM_1
+ROTARY_01
 Text Notes 1450 1900 2    60   ~ 0
-TRIM_10
+ROTARY_10
 Text Notes 1450 1800 2    60   ~ 0
-TRIM_9
+ROTARY_09
 Text Notes 1450 600  2    60   ~ 0
 H_RIGHT_JOYSTICK
@@
 V_RIGHT_JOYSTICK
 Text Notes 1450 2000 2    60   ~ 0
-TRIM_11
+ROTARY_11
 Text Notes 1450 2100 2    60   ~ 0
-TRIM_12
+ROTARY_12
 Text Notes 1450 800  2    60   ~ 0
 H_LEFT_JOYSTICK
@@
 $EndComp
 $Comp
-L RCTX-rescue:R_Network09-device RR2
-U 1 1 4EB6A2D0
-P 9600 5950
-F 0 "RR2" H 9350 6150 70  0000 C CNN
-F 1 "15K" H 9600 6150 70  0000 C CNN
-F 2 "Resistors_THT:R_Array_SIP10" H 9600 5950 60  0001 C CNN
-F 3 "" H 9600 5950 60  0001 C CNN
-	1    9600 5950
-	1    0    0    1
-$EndComp
-$Comp
 L RCTX-rescue:Conn_01x09-conn P16
 U 1 1 4EB6A357
@@
 $EndComp
 $Comp
-L RCTX-rescue:R_Network08-device RR1
-U 1 1 5F32EC78
-P 8800 5950
-F 0 "RR1" H 8650 6150 70  0000 R CNN
-F 1 "15k" H 8900 6150 70  0000 R CNN
-F 2 "Resistors_THT:R_Array_SIP9" V 9375 5950 50  0001 C CNN
-F 3 "http://www.vishay.com/docs/31509/csc.pdf" H 8800 5950 50  0001 C CNN
-	1    8800 5950
-	1    0    0    1
-$EndComp
-$Comp
 L RCTX-rescue:Conn_01x02-conn P12
 U 1 1 4C8B9793
@@
 Wire Wire Line
 	8400 1450 8400 2250
-Wire Wire Line
-	7400 5850 7150 5850
-Wire Wire Line
-	7400 6350 7400 5850
-Wire Wire Line
-	8400 6150 8400 6350
-Wire Wire Line
-	8400 6350 7900 6350
 Wire Wire Line
 	10100 6250 10100 6150
@@
 Wire Wire Line
 	7150 2250 8400 2250
-Connection ~ 8400 2250
-Wire Wire Line
-	8400 2250 8400 5750
 Wire Wire Line
 	8500 1450 8500 2350
@@
 Wire Wire Line
 	7150 2750 8700 2750
-Connection ~ 8700 2750
-Wire Wire Line
-	8700 2750 8700 5750
 Wire Wire Line
 	7150 2650 8600 2650
-Connection ~ 8600 2650
-Wire Wire Line
-	8600 2650 8600 5750
 Wire Wire Line
 	7150 2350 8500 2350
-Connection ~ 8500 2350
-Wire Wire Line
-	8500 2350 8500 5750
 $Comp
 L RCTX-rescue:Conn_01x04-conn P9
@@
 	2150 3550 1950 3550
 Connection ~ 2150 2750
-NoConn ~ 7150 6050
 $Comp
 L RCTX-rescue:GND-power #PWR02
@@
 	0    -1   -1   0
 $EndComp
-$Comp
-L RCTX-rescue:+3.3V-power #PWR04
-U 1 1 5FA40E40
-P 7900 6150
-F 0 "#PWR04" H 7900 6000 50  0001 C CNN
-F 1 "+3.3V" H 7915 6323 50  0000 C CNN
-F 2 "" H 7900 6150 50  0001 C CNN
-F 3 "" H 7900 6150 50  0001 C CNN
-	1    7900 6150
-	1    0    0    -1
-$EndComp
 Wire Wire Line
 	7900 6150 7900 6350
@@
 Wire Wire Line
 	5150 6200 5150 6500
+$Comp
+L RCTX-rescue:R_Network09-device RR2
+U 1 1 4EB6A2D0
+P 9600 5950
+F 0 "RR2" H 9350 6150 70  0000 C CNN
+F 1 "15K" H 9600 6150 70  0000 C CNN
+F 2 "Resistors_THT:R_Array_SIP10" H 9600 5950 60  0001 C CNN
+F 3 "" H 9600 5950 60  0001 C CNN
+	1    9600 5950
+	1    0    0    1
+$EndComp
+Wire Wire Line
+	7400 6350 7400 6050
+NoConn ~ 7150 5850
+Wire Wire Line
+	8400 6350 7900 6350
+Wire Wire Line
+	8400 6150 8400 6350
+$Comp
+L RCTX-rescue:R_Network08-device RR1
+U 1 1 5F32EC78
+P 8800 5950
+F 0 "RR1" H 8650 6150 70  0000 R CNN
+F 1 "15k" H 8900 6150 70  0000 R CNN
+F 2 "Resistors_THT:R_Array_SIP9" V 9375 5950 50  0001 C CNN
+F 3 "http://www.vishay.com/docs/31509/csc.pdf" H 8800 5950 50  0001 C CNN
+	1    8800 5950
+	1    0    0    1
+$EndComp
+Connection ~ 8400 2250
+Wire Wire Line
+	8400 2250 8400 5750
+Connection ~ 8500 2350
+Wire Wire Line
+	8500 2350 8500 5750
+Connection ~ 8600 2650
+Wire Wire Line
+	8600 2650 8600 5750
+Connection ~ 8700 2750
+Wire Wire Line
+	8700 2750 8700 5750
+Wire Wire Line
+	7400 6050 7150 6050
+$Comp
+L RCTX-rescue:GND-power #PWR?
+U 1 1 5F437E7A
+P 7900 6150
+F 0 "#PWR?" H 7900 5900 50  0001 C CNN
+F 1 "GND" H 7900 6000 50  0000 C CNN
+F 2 "" H 7900 6150 50  0001 C CNN
+F 3 "" H 7900 6150 50  0001 C CNN
+	1    7900 6150
+	-1   0    0    1
+$EndComp
 $EndSCHEMATC
