File: kicad/RCTX_JA.sch (KiCad schematic (older format))
At the start: 31 parts, among them J1 ROTARY_4, J10 H_RIGHT_JOYSTIC, J11 ROTARY_9, J12 V_RIGHT_JOYSTIC, J13 ROTARY_10, J14 H_LEFT_JOYSTIC, J15 ROTARY_11, J16 V_LEFT_JOYSTIC, J17 ROTARY_12, J18 MULTI_PROP_1, J19 MULTI_PROP_2, J2 ROTARY_5, J3 ROTARY_3, J4 ROTARY_6, J5 ROTARY_2, J6 ROTARY_7, J7 ROTARY_1, J8 ROTARY_8, J9 PWR_BUS, U3 LM324, U4 LM324, U5 LM324, U6 LM324

Commit message: Adding 5110 display
Parts:
- added C?: 100nF, symbol device:C
- added C?: 1uF, symbol device:CP
- added R?: 150, symbol device:R
- added R?: 470, symbol device:R
- added U?: LM117_TO3, TO_SOT_Packages_THT:TO-3, symbol regul:LM117_TO3
- J9: symbol conn:Conn_01x05 -> conn:Conn_01x04
Connections:
- net GND: now reaches C10.2, C11.1, C12.1, C13.2, C6.2, C7.1, C8.1, C9.2, J1.1 (Pin_1), J10.1 (Pin_1), J11.1 (Pin_1), J12.1 (Pin_1), J13.1 (Pin_1), J14.1 (Pin_1), J15.1 (Pin_1), J16.1 (Pin_1), J17.1 (Pin_1), J2.1 (Pin_1), J3.1 (Pin_1), J4.1 (Pin_1), J5.1 (Pin_1), J6.1 (Pin_1), J7.1 (Pin_1), J8.1 (Pin_1), U3.11 (V-), U3.11 (V-), U3.11 (V-), U3.11 (V-), U4.11 (V-), U4.11 (V-), U4.11 (V-), U4.11 (V-), U5.11 (V-), U5.11 (V-), U5.11 (V-), U5.11 (V-), U6.11 (V-), U6.11 (V-), U6.11 (V-), U6.11 (V-)
- net GND: now also J9.3 (Pin_3), C?.2, C?.2, R?.1; no longer J9.4 (Pin_4)
- net at J1.3 (Pin_3), J11.3 (Pin_3), J13.3 (Pin_3)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: now also C?.1, R?.1, U?.3 (VO); no longer J9.1 (Pin_1)
- net +5V: now reaches C10.1, C11.2, C12.2, C13.1, C6.1, C7.2, C8.2, C9.1, U3.4 (V+), U3.4 (V+), U3.4 (V+), U3.4 (V+), U4.4 (V+), U4.4 (V+), U4.4 (V+), U4.4 (V+), U5.4 (V+), U5.4 (V+), U5.4 (V+), U5.4 (V+), U6.4 (V+), U6.4 (V+), U6.4 (V+), U6.4 (V+)
- net +5V: now also J9.2 (Pin_2); no longer J9.3 (Pin_3)
- net +3V3: now reaches J10.3 (Pin_3), J12.3 (Pin_3), J14.3 (Pin_3), J16.3 (Pin_3)
- net +3V3: now also J9.1 (Pin_1), C?.1, U?.2 (VI); no longer J9.2 (Pin_2)
- new net: R?.2, R?.2, U?.1 (ADJ)
Other:
- note removed: "+1.65V"
- moved on the sheet: C10, C11, C12, C13, C6, C7, C8, C9, J1, J10, J11, J12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

Commit message: Adding footprints
Parts:
- C10, C9: footprint (none) -> Capacitors_THT:CP_Radial_D5.0mm_P2.50mm; symbol device:CP -> RCTX-rescue:CP-device
- C11, C8: footprint (none) -> Capacitors_THT:C_Disc_D3.0mm_W1.6mm_P2.50mm; symbol device:C -> RCTX-rescue:C-device
- C12: renamed from C?; footprint (none) -> Capacitors_THT:C_Disc_D3.0mm_W1.6mm_P2.50mm; symbol device:C -> RCTX-rescue:C-device
- C13: renamed from C12; footprint (none) -> Capacitors_THT:C_Disc_D3.0mm_W1.6mm_P2.50mm; symbol device:C -> RCTX-rescue:C-device
- C14: renamed from C13; footprint (none) -> Capacitors_THT:CP_Radial_D5.0mm_P2.50mm; symbol device:CP -> RCTX-rescue:CP-device
- C5: renamed from C6; footprint (none) -> Capacitors_THT:CP_Radial_D5.0mm_P2.50mm; symbol device:CP -> RCTX-rescue:CP-device
- C6: renamed from C7; footprint (none) -> Capacitors_THT:C_Disc_D3.0mm_W1.6mm_P2.50mm; symbol device:C -> RCTX-rescue:C-device
- C7: renamed from C?; footprint (none) -> Capacitors_THT:CP_Radial_D5.0mm_P2.50mm; symbol device:CP -> RCTX-rescue:CP-device
- J1, J10, J11, J12, J13, J14, J15, J16, J17, J2, J3, J4, J5, J6, J7, J8: footprint (none) -> servo_conn:SRV_1; symbol conn:Conn_01x03 -> RCTX-rescue:Conn_01x03-conn
- J18, J19: footprint (none) -> Connectors_Samtec:SL-108-X-XX_1x08; symbol conn:Conn_01x08 -> RCTX-rescue:Conn_01x08-conn
- J9: footprint (none) -> Connectors_Samtec:SL-104-X-XX_1x04; symbol conn:Conn_01x04 -> RCTX-rescue:Conn_01x04-conn
- R3, R4: renamed from R?; footprint (none) -> Resistors_THT:R_Axial_DIN0204_L3.6mm_D1.6mm_P1.90mm_Vertical; symbol device:R -> RCTX-rescue:R-device
- U3, U4: footprint (none) -> Housings_DIP:DIP-14_W7.62mm; symbol linear:LM324 -> RCTX-rescue:LM324-linear
- U5: renamed from U?; footprint TO_SOT_Packages_THT:TO-3 -> TO_SOT_Packages_THT:TO-92_Inline_Narrow_Oval; symbol regul:LM117_TO3 -> RCTX-rescue:LM117_TO3-regul
- U6: renamed from U5; footprint (none) -> Housings_DIP:DIP-14_W7.62mm; symbol linear:LM324 -> RCTX-rescue:LM324-linear
- U7: renamed from U6; footprint (none) -> Housings_DIP:DIP-14_W7.62mm; symbol linear:LM324 -> RCTX-rescue:LM324-linear
