File: kicad/RCTX_JA.sch (KiCad schematic (older format))
At the start: 36 parts, among them J1 ROTARY_4, J10 H_RIGHT_JOYSTIC, J11 ROTARY_9, J12 V_RIGHT_JOYSTIC, J13 ROTARY_10, J14 H_LEFT_JOYSTIC, J15 ROTARY_11, J16 V_LEFT_JOYSTIC, J17 ROTARY_12, J18 MULTI_PROP_1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

Commit message: renaming switches, buttons and trims
Other:
- note added: "ROTARY_01"
- note added: "ROTARY_02"
- note added: "ROTARY_03"
- note added: "ROTARY_04"
- note added: "ROTARY_05"
- note added: "ROTARY_06"
- note added: "ROTARY_07"
- note added: "ROTARY_08"
- note added: "ROTARY_09"
- note added: "ROTARY_10"
- note added: "ROTARY_11"
- note added: "ROTARY_12"
- note removed: "TRIM_1"
- note removed: "TRIM_10"
- note removed: "TRIM_11"
- note removed: "TRIM_12"
- note removed: "TRIM_2"
- note removed: "TRIM_3"
- note removed: "TRIM_4"
- note removed: "TRIM_5"
- note removed: "TRIM_6"
- note removed: "TRIM_7"
- note removed: "TRIM_8"
- note removed: "TRIM_9"
Changed lines of the file:
@@
 	9450 4800 9450 5500
 Text Notes 10700 2250 1    50   ~ 0
-TRIM_1
+ROTARY_01
 Text Notes 10800 2250 1    50   ~ 0
-TRIM_2
+ROTARY_02
 Text Notes 10900 2250 1    50   ~ 0
-TRIM_3
+ROTARY_03
 Text Notes 11000 2250 1    50   ~ 0
-TRIM_4
-Text Notes 10350 5100 1    50   ~ 0
-TRIM_5
-Text Notes 10450 5100 1    50   ~ 0
-TRIM_6
-Text Notes 10550 5100 1    50   ~ 0
-TRIM_7
-Text Notes 10650 5100 1    50   ~ 0
-TRIM_8
-Text Notes 10750 5100 1    50   ~ 0
-TRIM_9
-Text Notes 10850 5100 1    50   ~ 0
-TRIM_10
-Text Notes 10950 5100 1    50   ~ 0
-TRIM_11
-Text Notes 11050 5100 1    50   ~ 0
-TRIM_12
+ROTARY_04
+Text Notes 10350 5200 1    50   ~ 0
+ROTARY_05
+Text Notes 10450 5200 1    50   ~ 0
+ROTARY_06
+Text Notes 10550 5200 1    50   ~ 0
+ROTARY_07
+Text Notes 10650 5200 1    50   ~ 0
+ROTARY_08
+Text Notes 10750 5200 1    50   ~ 0
+ROTARY_09
+Text Notes 10850 5200 1    50   ~ 0
+ROTARY_10
+Text Notes 10950 5200 1    50   ~ 0
+ROTARY_11
+Text Notes 11050 5200 1    50   ~ 0
+ROTARY_12
 $Comp
 L conn:Conn_01x04 J9
