File: kicad/RCTX_KPD.sch (KiCad schematic (older format))
At the start: 27 parts, among them P35 KEYBOARD, SW23 SPST, SW24 SPST, SW25 SPST, SW26 SPST, SW27 SPST, SW28 SPST, SW29 SPST, SW30 SPST, SW31 CODING_SWITCH, SW32 CODING_SWITCH

Commit message: Adding 5110 display
Parts:
- renumbered SW23 to SW24, SW24 to SW25, SW25 to SW26, SW26 to SW27, SW27 to SW28, SW28 to SW29, SW29 to SW30, SW30 to SW31, SW31 to SW32, SW32 to SW33
Other:
- moved on the sheet: SW27, SW28, SW29, SW30, SW31
Changed lines of the file:
@@
 Connection ~ 5450 2300
 Wire Wire Line
-	5750 2700 5750 2300
-Wire Wire Line
-	5150 2300 5150 2700
-Wire Wire Line
-	4850 2300 4850 2700
+	5750 2750 5750 2300
+Wire Wire Line
+	5150 2300 5150 2750
+Wire Wire Line
+	4850 2300 4850 2750
 Connection ~ 3950 2400
 Wire Wire Line
@@
 	4250 4050 4250 3150
 Wire Wire Line
-	4850 4050 4850 3100
-Wire Wire Line
-	5450 4050 5450 3100
+	4850 4050 4850 3150
+Wire Wire Line
+	5450 4050 5450 3150
 Wire Wire Line
 	6100 4050 6100 3400
@@
 	6200 3400 6200 4450
 Wire Wire Line
-	5750 3100 5750 4050
-Wire Wire Line
-	5150 3100 5150 4050
+	5750 3150 5750 4050
+Wire Wire Line
+	5150 3150 5150 4050
 Wire Wire Line
 	3950 3150 3950 4050
@@
 	3950 2400 3950 2750
 Wire Wire Line
-	4550 2700 4550 2400
+	4550 2750 4550 2400
 Connection ~ 4250 2400
 Wire Wire Line
-	5450 2700 5450 2300
+	5450 2750 5450 2300
 Connection ~ 5150 2300
 Wire Wire Line
@@
 $EndComp
 $Comp
+L switches:SW_Push SW31
+U 1 1 4EAF0E37
+P 5750 2950
+F 0 "SW31" H 5400 2850 70  0000 C CNN
+F 1 "SPST" H 6100 2850 70  0000 C CNN
+F 2 "" H 5750 2950 50  0001 C CNN
+F 3 "" H 5750 2950 50  0001 C CNN
+	1    5750 2950
+	0    -1   -1   0
+$EndComp
+$Comp
 L switches:SW_Push SW30
-U 1 1 4EAF0E37
-P 5750 2900
-F 0 "SW30" H 5400 2800 70  0000 C CNN
-F 1 "SPST" H 6100 2800 70  0000 C CNN
-F 2 "" H 5750 2900 50  0001 C CNN
-F 3 "" H 5750 2900 50  0001 C CNN
-	1    5750 2900
+U 1 1 4EAF0E34
+P 5450 2950
+F 0 "SW30" H 5100 2850 70  0000 C CNN
+F 1 "SPST" H 5800 2850 70  0000 C CNN
+F 2 "" H 5450 2950 50  0001 C CNN
+F 3 "" H 5450 2950 50  0001 C CNN
+	1    5450 2950
 	0    -1   -1   0
 $EndComp
 $Comp
 L switches:SW_Push SW29
-U 1 1 4EAF0E34
-P 5450 2900
-F 0 "SW29" H 5100 2800 70  0000 C CNN
-F 1 "SPST" H 5800 2800 70  0000 C CNN
-F 2 "" H 5450 2900 50  0001 C CNN
-F 3 "" H 5450 2900 50  0001 C CNN
-	1    5450 2900
+U 1 1 4EAF0E31
+P 5150 2950
+F 0 "SW29" H 4800 2850 70  0000 C CNN
+F 1 "SPST" H 5500 2850 70  0000 C CNN
+F 2 "" H 5150 2950 50  0001 C CNN
+F 3 "" H 5150 2950 50  0001 C CNN
+	1    5150 2950
 	0    -1   -1   0
 $EndComp
 $Comp
 L switches:SW_Push SW28
-U 1 1 4EAF0E31
-P 5150 2900
-F 0 "SW28" H 4800 2800 70  0000 C CNN
-F 1 "SPST" H 5500 2800 70  0000 C CNN
-F 2 "" H 5150 2900 50  0001 C CNN
-F 3 "" H 5150 2900 50  0001 C CNN
-	1    5150 2900
+U 1 1 4EAF0E2E
+P 4850 2950
+F 0 "SW28" H 4500 2850 70  0000 C CNN
+F 1 "SPST" H 5200 2850 70  0000 C CNN
+F 2 "" H 4850 2950 50  0001 C CNN
+F 3 "" H 4850 2950 50  0001 C CNN
+	1    4850 2950
 	0    -1   -1   0
 $EndComp
 $Comp
 L switches:SW_Push SW27
-U 1 1 4EAF0E2E
-P 4850 2900
-F 0 "SW27" H 4500 2800 70  0000 C CNN
-F 1 "SPST" H 5200 2800 70  0000 C CNN
-F 2 "" H 4850 2900 50  0001 C CNN
-F 3 "" H 4850 2900 50  0001 C CNN
-	1    4850 2900
+U 1 1 4EAF0E2B
+P 4550 2950
+F 0 "SW27" H 4200 2850 70  0000 C CNN
+F 1 "SPST" H 4900 2850 70  0000 C CNN
+F 2 "" H 4550 2950 50  0001 C CNN
+F 3 "" H 4550 2950 50  0001 C CNN
+	1    4550 2950
 	0    -1   -1   0
 $EndComp
 $Comp
 L switches:SW_Push SW26
-U 1 1 4EAF0E2B
-P 4550 2900
-F 0 "SW26" H 4200 2800 70  0000 C CNN
-F 1 "SPST" H 4900 2800 70  0000 C CNN
-F 2 "" H 4550 2900 50  0001 C CNN
-F 3 "" H 4550 2900 50  0001 C CNN
-	1    4550 2900
-	0    -1   -1   0
-$EndComp
-$Comp
-L switches:SW_Push SW25
 U 1 1 4EAF0E29
 P 4250 2950
-F 0 "SW25" H 3900 2850 70  0000 C CNN
+F 0 "SW26" H 3900 2850 70  0000 C CNN
 F 1 "SPST" H 4600 2850 70  0000 C CNN
 F 2 "" H 4250 2950 50  0001 C CNN
@@
 $EndComp
 $Comp
-L switches:SW_Push SW24
+L switches:SW_Push SW25
 U 1 1 4EAF0E27
 P 3950 2950
-F 0 "SW24" H 3600 2850 70  0000 C CNN
+F 0 "SW25" H 3600 2850 70  0000 C CNN
 F 1 "SPST" H 4300 2850 70  0000 C CNN
 F 2 "" H 3950 2950 50  0001 C CNN
@@
 $EndComp
 $Comp
-L switches:SW_Coded SW32
+L switches:SW_Coded SW33
 U 1 1 4CA2397F
 P 7200 2900
-F 0 "SW32" H 7300 3250 60  0000 C CNN
+F 0 "SW33" H 7300 3250 60  0000 C CNN
 F 1 "CODING_SWITCH" V 6850 2900 60  0000 C CNN
 F 2 "" H 7200 2900 50  0001 C CNN
@@
 $EndComp
 $Comp
-L switches:SW_Coded SW31
+L switches:SW_Coded SW32
 U 1 1 4CA23972
 P 6300 2900
-F 0 "SW31" H 6400 3250 60  0000 C CNN
+F 0 "SW32" H 6400 3250 60  0000 C CNN
 F 1 "CODING_SWITCH" V 5950 2950 60  0000 C CNN
 F 2 "" H 6300 2900 50  0001 C CNN
@@
 $EndComp
 $Comp
-L switches:SW_Push SW23
+L switches:SW_Push SW24
 U 1 1 4CA23920
 P 3650 2950
-F 0 "SW23" H 3300 2850 70  0000 C CNN
+F 0 "SW24" H 3300 2850 70  0000 C CNN
 F 1 "SPST" H 4000 2850 70  0000 C CNN
 F 2 "" H 3650 2950 50  0001 C CNN
@@
 	4250 6050 5450 6050
 Wire Wire Line
-	4550 3100 4550 4050
+	4550 3150 4550 4050
 $Comp
 L device:D D41

Commit message: Adding footprints
Parts:
- D38, D39, D40, D41, D42, D43, D44, D45, D46, D47, D48, D49, D50, D51, D52, D53: footprint (none) -> Diodes_THT:D_5W_P5.08mm_Vertical_KathodeUp; symbol device:D -> RCTX-rescue:D-device
- P39: renamed from P35; footprint (none) -> Connectors_Samtec:SL-108-X-XX_1x08; symbol conn:Conn_01x08 -> RCTX-rescue:Conn_01x08-conn
- SW25: renamed from SW24; footprint (none) -> Buttons_Switches_THT:SW_PUSH_6mm_h5mm; symbol switches:SW_Push -> RCTX-rescue:SW_Push-switches
- SW26: renamed from SW25; footprint (none) -> Buttons_Switches_THT:SW_PUSH_6mm_h5mm; symbol switches:SW_Push -> RCTX-rescue:SW_Push-switches
- SW27: renamed from SW26; footprint (none) -> Buttons_Switches_THT:SW_PUSH_6mm_h5mm; symbol switches:SW_Push -> RCTX-rescue:SW_Push-switches
- SW28: renamed from SW27; footprint (none) -> Buttons_Switches_THT:SW_PUSH_6mm_h5mm; symbol switches:SW_Push -> RCTX-rescue:SW_Push-switches
- SW29: renamed from SW28; footprint (none) -> Buttons_Switches_THT:SW_PUSH_6mm_h5mm; symbol switches:SW_Push -> RCTX-rescue:SW_Push-switches
- SW30: renamed from SW29; footprint (none) -> Buttons_Switches_THT:SW_PUSH_6mm_h5mm; symbol switches:SW_Push -> RCTX-rescue:SW_Push-switches
- SW31: renamed from SW30; footprint (none) -> Buttons_Switches_THT:SW_PUSH_6mm_h5mm; symbol switches:SW_Push -> RCTX-rescue:SW_Push-switches
- SW32: renamed from SW31; footprint (none) -> Buttons_Switches_THT:SW_PUSH_6mm_h5mm; symbol switches:SW_Push -> RCTX-rescue:SW_Push-switches
- SW33: renamed from SW32; footprint (none) -> Buttons_Switches_THT:Nidec_Copal_SH-7010C; symbol switches:SW_Coded -> RCTX-rescue:SW_Coded-switches
- SW34: renamed from SW33; footprint (none) -> Buttons_Switches_THT:Nidec_Copal_SH-7010C; symbol switches:SW_Coded -> RCTX-rescue:SW_Coded-switches
Changed lines of the file:
@@
 Connection ~ 4250 6050
 $Comp
-L conn:Conn_01x08 P35
+L RCTX-rescue:Conn_01x08-conn P39
 U 1 1 4EB6A839
 P 2150 5750
-F 0 "P35" H 2150 5250 60  0000 C CNN
+F 0 "P39" H 2150 5250 60  0000 C CNN
 F 1 "KEYBOARD" V 2250 5750 60  0000 C CNN
-F 2 "" H 2150 5750 50  0001 C CNN
+F 2 "Connectors_Samtec:SL-108-X-XX_1x08" H 2150 5750 50  0001 C CNN
 F 3 "" H 2150 5750 50  0001 C CNN
 	1    2150 5750
@@
 $EndComp
 $Comp
-L switches:SW_Push SW31
+L RCTX-rescue:SW_Push-switches SW32
 U 1 1 4EAF0E37
 P 5750 2950
-F 0 "SW31" H 5400 2850 70  0000 C CNN
+F 0 "SW32" H 5400 2850 70  0000 C CNN
 F 1 "SPST" H 6100 2850 70  0000 C CNN
-F 2 "" H 5750 2950 50  0001 C CNN
+F 2 "Buttons_Switches_THT:SW_PUSH_6mm_h5mm" H 5750 2950 50  0001 C CNN
 F 3 "" H 5750 2950 50  0001 C CNN
 	1    5750 2950
@@
 $EndComp
 $Comp
-L switches:SW_Push SW30
+L RCTX-rescue:SW_Push-switches SW31
 U 1 1 4EAF0E34
 P 5450 2950
-F 0 "SW30" H 5100 2850 70  0000 C CNN
+F 0 "SW31" H 5100 2850 70  0000 C CNN
 F 1 "SPST" H 5800 2850 70  0000 C CNN
-F 2 "" H 5450 2950 50  0001 C CNN
+F 2 "Buttons_Switches_THT:SW_PUSH_6mm_h5mm" H 5450 2950 50  0001 C CNN
 F 3 "" H 5450 2950 50  0001 C CNN
 	1    5450 2950
@@
 $EndComp
 $Comp
-L switches:SW_Push SW29
+L RCTX-rescue:SW_Push-switches SW30
 U 1 1 4EAF0E31
 P 5150 2950
-F 0 "SW29" H 4800 2850 70  0000 C CNN
+F 0 "SW30" H 4800 2850 70  0000 C CNN
 F 1 "SPST" H 5500 2850 70  0000 C CNN
-F 2 "" H 5150 2950 50  0001 C CNN
+F 2 "Buttons_Switches_THT:SW_PUSH_6mm_h5mm" H 5150 2950 50  0001 C CNN
 F 3 "" H 5150 2950 50  0001 C CNN
 	1    5150 2950
@@
 $EndComp
 $Comp
-L switches:SW_Push SW28
+L RCTX-rescue:SW_Push-switches SW29
 U 1 1 4EAF0E2E
 P 4850 2950
-F 0 "SW28" H 4500 2850 70  0000 C CNN
+F 0 "SW29" H 4500 2850 70  0000 C CNN
 F 1 "SPST" H 5200 2850 70  0000 C CNN
-F 2 "" H 4850 2950 50  0001 C CNN
+F 2 "Buttons_Switches_THT:SW_PUSH_6mm_h5mm" H 4850 2950 50  0001 C CNN
 F 3 "" H 4850 2950 50  0001 C CNN
 	1    4850 2950
@@
 $EndComp
 $Comp
-L switches:SW_Push SW27
+L RCTX-rescue:SW_Push-switches SW28
 U 1 1 4EAF0E2B
 P 4550 2950
-F 0 "SW27" H 4200 2850 70  0000 C CNN
+F 0 "SW28" H 4200 2850 70  0000 C CNN
 F 1 "SPST" H 4900 2850 70  0000 C CNN
-F 2 "" H 4550 2950 50  0001 C CNN
+F 2 "Buttons_Switches_THT:SW_PUSH_6mm_h5mm" H 4550 2950 50  0001 C CNN
 F 3 "" H 4550 2950 50  0001 C CNN
 	1    4550 2950
@@
 $EndComp
 $Comp
-L switches:SW_Push SW26
+L RCTX-rescue:SW_Push-switches SW27
 U 1 1 4EAF0E29
 P 4250 2950
-F 0 "SW26" H 3900 2850 70  0000 C CNN
+F 0 "SW27" H 3900 2850 70  0000 C CNN
 F 1 "SPST" H 4600 2850 70  0000 C CNN
-F 2 "" H 4250 2950 50  0001 C CNN
+F 2 "Buttons_Switches_THT:SW_PUSH_6mm_h5mm" H 4250 2950 50  0001 C CNN
 F 3 "" H 4250 2950 50  0001 C CNN
 	1    4250 2950
@@
 $EndComp
 $Comp
-L switches:SW_Push SW25
+L RCTX-rescue:SW_Push-switches SW26
 U 1 1 4EAF0E27
 P 3950 2950
-F 0 "SW25" H 3600 2850 70  0000 C CNN
+F 0 "SW26" H 3600 2850 70  0000 C CNN
 F 1 "SPST" H 4300 2850 70  0000 C CNN
-F 2 "" H 3950 2950 50  0001 C CNN
+F 2 "Buttons_Switches_THT:SW_PUSH_6mm_h5mm" H 3950 2950 50  0001 C CNN
 F 3 "" H 3950 2950 50  0001 C CNN
 	1    3950 2950
@@
 $EndComp
 $Comp
-L device:D D53
+L RCTX-rescue:D-device D53
 U 1 1 4EAF0DF5
 P 7300 4600
 F 0 "D53" H 7150 4650 40  0000 C CNN
 F 1 "1N4148" H 7500 4650 40  0000 C CNN
-F 2 "" H 7300 4600 50  0001 C CNN
+F 2 "Diodes_THT:D_5W_P5.08mm_Vertical_KathodeUp" H 7300 4600 50  0001 C CNN
 F 3 "" H 7300 4600 50  0001 C CNN
 	1    7300 4600
@@
 $EndComp
 $Comp
-L device:D D52
+L RCTX-rescue:D-device D52
 U 1 1 4EAF0DF3
 P 7200 4200
 F 0 "D52" H 7050 4250 40  0000 C CNN
 F 1 "1N4148" H 7400 4250 40  0000 C CNN
-F 2 "" H 7200 4200 50  0001 C CNN
+F 2 "Diodes_THT:D_5W_P5.08mm_Vertical_KathodeUp" H 7200 4200 50  0001 C CNN
 F 3 "" H 7200 4200 50  0001 C CNN
 	1    7200 4200
@@
 $EndComp
 $Comp
-L device:D D51
+L RCTX-rescue:D-device D51
 U 1 1 4EAF0DF1
 P 7100 4600
 F 0 "D51" H 6950 4650 40  0000 C CNN
 F 1 "1N4148" H 7300 4650 40  0000 C CNN
-F 2 "" H 7100 4600 50  0001 C CNN
+F 2 "Diodes_THT:D_5W_P5.08mm_Vertical_KathodeUp" H 7100 4600 50  0001 C CNN
 F 3 "" H 7100 4600 50  0001 C CNN
 	1    7100 4600
@@
 $EndComp
 $Comp
-L device:D D50
+L RCTX-rescue:D-device D50
 U 1 1 4EAF0DEF
 P 7000 4200
 F 0 "D50" H 6850 4250 40  0000 C CNN
 F 1 "1N4148" H 7200 4250 40  0000 C CNN
-F 2 "" H 7000 4200 50  0001 C CNN
+F 2 "Diodes_THT:D_5W_P5.08mm_Vertical_KathodeUp" H 7000 4200 50  0001 C CNN
 F 3 "" H 7000 4200 50  0001 C CNN
 	1    7000 4200
@@
 $EndComp
 $Comp
-L device:D D49
+L RCTX-rescue:D-device D49
 U 1 1 4EAF0DED
 P 6400 4600
 F 0 "D49" H 6250 4650 40  0000 C CNN
 F 1 "1N4148" H 6600 4650 40  0000 C CNN
-F 2 "" H 6400 4600 50  0001 C CNN
+F 2 "Diodes_THT:D_5W_P5.08mm_Vertical_KathodeUp" H 6400 4600 50  0001 C CNN
 F 3 "" H 6400 4600 50  0001 C CNN
 	1    6400 4600
@@
 $EndComp
 $Comp
-L device:D D48
+L RCTX-rescue:D-device D48
 U 1 1 4EAF0DEA
 P 6300 4200
 F 0 "D48" H 6150 4250 40  0000 C CNN
 F 1 "1N4148" H 6500 4250 40  0000 C CNN
-F 2 "" H 6300 4200 50  0001 C CNN
+F 2 "Diodes_THT:D_5W_P5.08mm_Vertical_KathodeUp" H 6300 4200 50  0001 C CNN
 F 3 "" H 6300 4200 50  0001 C CNN
 	1    6300 4200
@@
 $EndComp
 $Comp
-L device:D D47
+L RCTX-rescue:D-device D47
 U 1 1 4EAF0DE8
 P 6200 4600
 F 0 "D47" H 6050 4650 40  0000 C CNN
 F 1 "1N4148" H 6400 4650 40  0000 C CNN
-F 2 "" H 6200 4600 50  0001 C CNN
+F 2 "Diodes_THT:D_5W_P5.08mm_Vertical_KathodeUp" H 6200 4600 50  0001 C CNN
 F 3 "" H 6200 4600 50  0001 C CNN
 	1    6200 4600
@@
 $EndComp
 $Comp
-L device:D D46
+L RCTX-rescue:D-device D46
 U 1 1 4EAF0DE6
 P 6100 4200
 F 0 "D46" H 5950 4250 40  0000 C CNN
 F 1 "1N4148" H 6300 4250 40  0000 C CNN
-F 2 "" H 6100 4200 50  0001 C CNN
+F 2 "Diodes_THT:D_5W_P5.08mm_Vertical_KathodeUp" H 6100 4200 50  0001 C CNN
 F 3 "" H 6100 4200 50  0001 C CNN
 	1    6100 4200
@@
 $EndComp
 $Comp
-L device:D D45
+L RCTX-rescue:D-device D45
 U 1 1 4EAF0DE5
 P 5750 4200
 F 0 "D45" H 5600 4250 40  0000 C CNN
 F 1 "1N4148" H 5950 4250 40  0000 C CNN
-F 2 "" H 5750 4200 50  0001 C CNN
+F 2 "Diodes_THT:D_5W_P5.08mm_Vertical_KathodeUp" H 5750 4200 50  0001 C CNN
 F 3 "" H 5750 4200 50  0001 C CNN
 	1    5750 4200
@@
 $EndComp
 $Comp
-L device:D D44
+L RCTX-rescue:D-device D44
 U 1 1 4EAF0DE3
 P 5450 4200
 F 0 "D44" H 5300 4250 40  0000 C CNN
 F 1 "1N4148" H 5650 4250 40  0000 C CNN
-F 2 "" H 5450 4200 50  0001 C CNN
+F 2 "Diodes_THT:D_5W_P5.08mm_Vertical_KathodeUp" H 5450 4200 50  0001 C CNN
 F 3 "" H 5450 4200 50  0001 C CNN
 	1    5450 4200
@@
 $EndComp
 $Comp
-L device:D D43
+L RCTX-rescue:D-device D43
 U 1 1 4EAF0DE0
 P 5150 4200
 F 0 "D43" H 5000 4250 40  0000 C CNN
 F 1 "1N4148" H 5350 4250 40  0000 C CNN
-F 2 "" H 5150 4200 50  0001 C CNN
+F 2 "Diodes_THT:D_5W_P5.08mm_Vertical_KathodeUp" H 5150 4200 50  0001 C CNN
 F 3 "" H 5150 4200 50  0001 C CNN
 	1    5150 4200
@@
 $EndComp
 $Comp
-L device:D D40
+L RCTX-rescue:D-device D40
 U 1 1 4EAF0DD9
 P 4250 4200
 F 0 "D40" H 4100 4250 40  0000 C CNN
 F 1 "1N4148" H 4450 4250 40  0000 C CNN
-F 2 "" H 4250 4200 50  0001 C CNN
+F 2 "Diodes_THT:D_5W_P5.08mm_Vertical_KathodeUp" H 4250 4200 50  0001 C CNN
 F 3 "" H 4250 4200 50  0001 C CNN
 	1    4250 4200
@@
 $EndComp
 $Comp
-L device:D D39
+L RCTX-rescue:D-device D39
 U 1 1 4EAF0DD7
 P 3950 4200
 F 0 "D39" H 3800 4250 40  0000 C CNN
 F 1 "1N4148" H 4150 4250 40  0000 C CNN
-F 2 "" H 3950 4200 50  0001 C CNN
+F 2 "Diodes_THT:D_5W_P5.08mm_Vertical_KathodeUp" H 3950 4200 50  0001 C CNN
 F 3 "" H 3950 4200 50  0001 C CNN
 	1    3950 4200
@@
 $EndComp
 $Comp
-L device:D D38
+L RCTX-rescue:D-device D38
 U 1 1 4CA239B0
 P 3650 4200
 F 0 "D38" H 3500 4250 40  0000 C CNN
 F 1 "1N4148" H 3850 4250 40  0000 C CNN
-F 2 "" H 3650 4200 50  0001 C CNN
+F 2 "Diodes_THT:D_5W_P5.08mm_Vertical_KathodeUp" H 3650 4200 50  0001 C CNN
 F 3 "" H 3650 4200 50  0001 C CNN
 	1    3650 4200
@@
 $EndComp
 $Comp
-L switches:SW_Coded SW33
+L RCTX-rescue:SW_Coded-switches SW34
 U 1 1 4CA2397F
 P 7200 2900
-F 0 "SW33" H 7300 3250 60  0000 C CNN
+F 0 "SW34" H 7300 3250 60  0000 C CNN
 F 1 "CODING_SWITCH" V 6850 2900 60  0000 C CNN
-F 2 "" H 7200 2900 50  0001 C CNN
+F 2 "Buttons_Switches_THT:Nidec_Copal_SH-7010C" H 7200 2900 50  0001 C CNN
 F 3 "" H 7200 2900 50  0001 C CNN
 	1    7200 2900
@@
 $EndComp
 $Comp
-L switches:SW_Coded SW32
+L RCTX-rescue:SW_Coded-switches SW33
 U 1 1 4CA23972
 P 6300 2900
-F 0 "SW32" H 6400 3250 60  0000 C CNN
+F 0 "SW33" H 6400 3250 60  0000 C CNN
 F 1 "CODING_SWITCH" V 5950 2950 60  0000 C CNN
-F 2 "" H 6300 2900 50  0001 C CNN
+F 2 "Buttons_Switches_THT:Nidec_Copal_SH-7010C" H 6300 2900 50  0001 C CNN
 F 3 "" H 6300 2900 50  0001 C CNN
 	1    6300 2900
@@
 $EndComp
 $Comp
-L switches:SW_Push SW24
+L RCTX-rescue:SW_Push-switches SW25
 U 1 1 4CA23920
 P 3650 2950
-F 0 "SW24" H 3300 2850 70  0000 C CNN
+F 0 "SW25" H 3300 2850 70  0000 C CNN
 F 1 "SPST" H 4000 2850 70  0000 C CNN
-F 2 "" H 3650 2950 50  0001 C CNN
+F 2 "Buttons_Switches_THT:SW_PUSH_6mm_h5mm" H 3650 2950 50  0001 C CNN
 F 3 "" H 3650 2950 50  0001 C CNN
 	1    3650 2950
@@
 	4550 3150 4550 4050
 $Comp
-L device:D D41
+L RCTX-rescue:D-device D41
 U 1 1 4EAF0DDC
 P 4550 4200
 F 0 "D41" H 4400 4250 40  0000 C CNN
 F 1 "1N4148" H 4750 4250 40  0000 C CNN
-F 2 "" H 4550 4200 50  0001 C CNN
+F 2 "Diodes_THT:D_5W_P5.08mm_Vertical_KathodeUp" H 4550 4200 50  0001 C CNN
 F 3 "" H 4550 4200 50  0001 C CNN
 	1    4550 4200
@@
 $EndComp
 $Comp
-L device:D D42
+L RCTX-rescue:D-device D42
 U 1 1 4EAF0DDE
 P 4850 4200
 F 0 "D42" H 4700 4250 40  0000 C CNN
 F 1 "1N4148" H 5050 4250 40  0000 C CNN
-F 2 "" H 4850 4200 50  0001 C CNN
+F 2 "Diodes_THT:D_5W_P5.08mm_Vertical_KathodeUp" H 4850 4200 50  0001 C CNN
 F 3 "" H 4850 4200 50  0001 C CNN
 	1    4850 4200
