File: kicad/RCTX_KPD.sch (KiCad schematic (older format))
At the start: 27 parts, among them P35 KEYBOARD, SW24 SPST, SW25 SPST, SW26 SPST, SW27 SPST, SW28 SPST, SW29 SPST, SW30 SPST, SW31 SPST, SW32 CODING_SWITCH, SW33 CODING_SWITCH

Commit message: renaming switches, buttons and trims
Parts:
- renumbered SW24 to BTN1, SW25 to BTN2, SW26 to BTN3, SW27 to BTN4, SW28 to BTN5, SW29 to BTN6, SW30 to BTN7, SW31 to BTN8
Changed lines of the file:
@@
 $EndComp
 $Comp
-L switches:SW_Push SW31
+L switches:SW_Push BTN8
 U 1 1 4EAF0E37
 P 5750 2950
-F 0 "SW31" H 5400 2850 70  0000 C CNN
+F 0 "BTN8" H 5400 2850 70  0000 C CNN
 F 1 "SPST" H 6100 2850 70  0000 C CNN
 F 2 "" H 5750 2950 50  0001 C CNN
@@
 $EndComp
 $Comp
-L switches:SW_Push SW30
+L switches:SW_Push BTN7
 U 1 1 4EAF0E34
 P 5450 2950
-F 0 "SW30" H 5100 2850 70  0000 C CNN
+F 0 "BTN7" H 5100 2850 70  0000 C CNN
 F 1 "SPST" H 5800 2850 70  0000 C CNN
 F 2 "" H 5450 2950 50  0001 C CNN
@@
 $EndComp
 $Comp
-L switches:SW_Push SW29
+L switches:SW_Push BTN6
 U 1 1 4EAF0E31
 P 5150 2950
-F 0 "SW29" H 4800 2850 70  0000 C CNN
+F 0 "BTN6" H 4800 2850 70  0000 C CNN
 F 1 "SPST" H 5500 2850 70  0000 C CNN
 F 2 "" H 5150 2950 50  0001 C CNN
@@
 $EndComp
 $Comp
-L switches:SW_Push SW28
+L switches:SW_Push BTN5
 U 1 1 4EAF0E2E
 P 4850 2950
-F 0 "SW28" H 4500 2850 70  0000 C CNN
+F 0 "BTN5" H 4500 2850 70  0000 C CNN
 F 1 "SPST" H 5200 2850 70  0000 C CNN
 F 2 "" H 4850 2950 50  0001 C CNN
@@
 $EndComp
 $Comp
-L switches:SW_Push SW27
+L switches:SW_Push BTN4
 U 1 1 4EAF0E2B
 P 4550 2950
-F 0 "SW27" H 4200 2850 70  0000 C CNN
+F 0 "BTN4" H 4200 2850 70  0000 C CNN
 F 1 "SPST" H 4900 2850 70  0000 C CNN
 F 2 "" H 4550 2950 50  0001 C CNN
@@
 $EndComp
 $Comp
-L switches:SW_Push SW26
+L switches:SW_Push BTN3
 U 1 1 4EAF0E29
 P 4250 2950
-F 0 "SW26" H 3900 2850 70  0000 C CNN
+F 0 "BTN3" H 3900 2850 70  0000 C CNN
 F 1 "SPST" H 4600 2850 70  0000 C CNN
 F 2 "" H 4250 2950 50  0001 C CNN
@@
 $EndComp
 $Comp
-L switches:SW_Push SW25
+L switches:SW_Push BTN2
 U 1 1 4EAF0E27
 P 3950 2950
-F 0 "SW25" H 3600 2850 70  0000 C CNN
+F 0 "BTN2" H 3600 2850 70  0000 C CNN
 F 1 "SPST" H 4300 2850 70  0000 C CNN
 F 2 "" H 3950 2950 50  0001 C CNN
@@
 $EndComp
 $Comp
-L switches:SW_Push SW24
+L switches:SW_Push BTN1
 U 1 1 4CA23920
 P 3650 2950
-F 0 "SW24" H 3300 2850 70  0000 C CNN
+F 0 "BTN1" H 3300 2850 70  0000 C CNN
 F 1 "SPST" H 4000 2850 70  0000 C CNN
 F 2 "" H 3650 2950 50  0001 C CNN
