File: kicad/RCTX_LEDS.sch (KiCad schematic (older format))
At the start: 48 parts, among them J20 Conn_01x17, J21 Conn_01x17, J22 Conn_01x17, J23 Conn_01x17, P29 PWR_BUS, P30 LEDs, P31 CONN_8, P32 CONN_8, P33 CONN_8, P34 CONN_8, U7 MAX6969, U8 MAX6969

Commit message: Adding 5110 display
Parts:
- removed P30: LEDs, symbol conn:Conn_01x06
- added P?: Nokia 5110 Display, symbol conn:Conn_01x08
- added P?: LEDs, symbol conn:Conn_01x04
- added P?: DISPLAY, symbol conn:Conn_01x05
- added SW?: LED_SWITCH, symbol switches:SW_SPST
- P29: symbol conn:Conn_01x05 -> conn:Conn_01x04
Connections:
- net labels added: +3.3V, GND
- wire segments 236 -> 246
Other:
- note added: "/CE"
- note added: "/PWM"
- note added: "/RESET"
- note added: "D/C"
- note added: "LED"
- note added: "VCC"
- note removed: "+1.65V"
- note removed: "/OE1"
- note removed: "/OE2"
- note removed: "SDO"
- note removed: "while (true)\n{\n uint32_t data = getDisplayData();\n /0E = 1;\n CLK = 0;\n DIN =1;\n for (int i=0; i<32; i++)\n {\n CLK = 1;\n /OE = !((data >> i) & 1);\n wait(PWM_ON_TIME);\n CLK = 0;\n DIN = 0;\n /OE = 1;\n }\n}"
- moved on the sheet: C14, C15, D10, D11, D12, D13, D14, D15, D16, D17, D18, D19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

Commit message: Adding footprints
Parts:
- C15: renamed from C14; footprint (none) -> Capacitors_THT:C_Disc_D3.0mm_W1.6mm_P2.50mm; symbol device:C -> RCTX-rescue:C-device
- C16: renamed from C15; footprint (none) -> Capacitors_THT:C_Disc_D3.0mm_W1.6mm_P2.50mm; symbol device:C -> RCTX-rescue:C-device
- D10, D11, D12, D13, D14, D15, D16, D17, D18, D19, D20, D21, D22, D23, D24, D25, D26, D27, D28, D29, D30, D31, D32, D33, D34, D35, D36, D37, D6, D7, D8, D9: footprint (none) -> LEDs:LED_D2.0mm_W4.0mm_H2.8mm_FlatTop; symbol device:LED -> RCTX-rescue:LED-device
- J20, J21, J22, J23: footprint (none) -> Connectors_Samtec:SL-117-X-XX_1x17; symbol conn:Conn_01x17 -> RCTX-rescue:Conn_01x17-conn
- P31: renamed from P29; footprint (none) -> Connectors_Samtec:SL-104-X-XX_1x04; symbol conn:Conn_01x04 -> RCTX-rescue:Conn_01x04-conn
- P32: renamed from P?; footprint (none) -> Connectors_Samtec:SL-104-X-XX_1x04; symbol conn:Conn_01x04 -> RCTX-rescue:Conn_01x04-conn
- P33: renamed from P?; footprint (none) -> Connectors_Samtec:SL-105-X-XX_1x05; symbol conn:Conn_01x05 -> RCTX-rescue:Conn_01x05-conn
- P34: renamed from P31; footprint (none) -> Connectors_Samtec:SL-108-X-XX_1x08; symbol conn:Conn_01x08 -> RCTX-rescue:Conn_01x08-conn
- P35: renamed from P32; footprint (none) -> Connectors_Samtec:SL-108-X-XX_1x08; symbol conn:Conn_01x08 -> RCTX-rescue:Conn_01x08-conn
- P36: renamed from P?; footprint (none) -> Connectors_Samtec:SL-108-X-XX_1x08; symbol conn:Conn_01x08 -> RCTX-rescue:Conn_01x08-conn
- P37: renamed from P33; footprint (none) -> Connectors_Samtec:SL-108-X-XX_1x08; symbol conn:Conn_01x08 -> RCTX-rescue:Conn_01x08-conn
- P38: renamed from P34; footprint (none) -> Connectors_Samtec:SL-108-X-XX_1x08; symbol conn:Conn_01x08 -> RCTX-rescue:Conn_01x08-conn
- R10: renamed from R9; footprint (none) -> Resistors_THT:R_Axial_DIN0204_L3.6mm_D1.6mm_P1.90mm_Vertical; symbol device:R -> RCTX-rescue:R-device
- R9: renamed from R8; footprint (none) -> Resistors_THT:R_Axial_DIN0204_L3.6mm_D1.6mm_P1.90mm_Vertical; symbol device:R -> RCTX-rescue:R-device
- SW24: renamed from SW?; footprint (none) -> Buttons_Switches_THT:SW_DIP_x1_W7.62mm_Slide_LowProfile; symbol switches:SW_SPST -> RCTX-rescue:SW_SPST-switches
- U8: renamed from U7; footprint (none) -> Housings_DIP:DIP-24_W7.62mm
- U9: renamed from U8; footprint (none) -> Housings_DIP:DIP-24_W7.62mm
