File: kicad/RCTX_MDL.sch (KiCad schematic (older format))
At the start: 39 parts, among them K1 CONN_3, P21 PWR_BUS, P22 TX_VCC, P23 MULTI_DIGITAL_1, P24 PWR_BUS, P25 CONN_4, P26 PWR_BUS, P27 MULTI_DIGITAL_2, P28 PWR_BUS, SW1 Reset, SW10 LEFT_3P1V, SW11 LEFT_3P1V, SW12 LEFT_3P1V, SW13 LEFT_3P1V, SW14 RIGHT_3P1V, SW15 RIGHT_3P1V, SW16 RIGHT_3P1V, SW17 RIGHT_3P1V, SW18 RIGHT_3P1V, SW19 RIGHT_3P1V, SW2 Program, SW20 RIGHT_3P1V, SW21 RIGHT_3P1V, SW22 RIGHT_3P1V, SW3 User, SW4 RF_SWITCH_3P2V, SW5 LEFT_3P2V, SW6 LEFT_3P1V, SW7 LEFT_3P1V, SW8 LEFT_3P1V, SW9 LEFT_3P1V

Commit message: Adding 5110 display
Parts:
- removed SW14: RIGHT_3P1V, symbol switches:SW_SPDT_MSM
- removed SW4: RF_SWITCH_3P2V, symbol switches:SW_SPDT_MSM
- removed SW5: LEFT_3P2V, symbol switches:SW_SPDT_MSM
- added SW14: RIGHT_3P2V_B, symbol switches:SW_SP3T
- added SW15: RIGHT_3P2V_A, symbol switches:SW_SP3T
- added SW4: RF_SWITCH_3P2V, symbol switches:SW_SP3T
- added SW5: LEFT_3P2V, symbol switches:SW_SP3T
- P21, P24, P26, P28: symbol conn:Conn_01x05 -> conn:Conn_01x04
- renumbered K1 to P1, SW15 to SW16, SW16 to SW17, SW17 to SW18, SW18 to SW19, SW19 to SW20, SW20 to SW21, SW21 to SW22, SW22 to SW23
Connections:
- net +3V3: now reaches SW10.1, SW11.1, SW12.1, SW13.1, SW6.1, SW7.1, SW8.1, SW9.1
- net +3V3: now also P21.3 (Pin_3), P24.1 (Pin_1), P24.3 (Pin_3), P26.1 (Pin_1), P28.1 (Pin_1), P28.3 (Pin_3), R4.2, R5.2, R6.2, R7.2, SW1.1 (A), SW10.3, SW11.3, SW12.3, SW13.3, SW16.1, SW16.3, SW17.1, SW17.3, SW18.1, SW18.3, SW19.1, SW19.3, SW2.1 (A), SW20.1, SW20.3, SW21.1, SW21.3, SW22.1, SW22.3, SW23.1, SW23.3, SW3.1 (A), SW6.3, SW7.3, SW8.3, SW9.3, SW15.1, SW15.4, SW5.1, SW5.4; no longer P24.2 (Pin_2)
- net at P23.1 (Pin_1): now also SW5.3
- net at P27.1 (Pin_1): now also SW15.3
- net at P22.2 (Pin_2): now also SW4.1
- net at P22.1 (Pin_1): now also SW4.3
- now unconnected: P21.4 (Pin_4), P24.4 (Pin_4), P26.2 (Pin_2), P28.2 (Pin_2), P28.4 (Pin_4)
- no-connect marks 15 -> 18
Other:
- note removed: "+1.65V"
Changed lines of the file:
@@
 U 1 1 4EB6D39A
 P 6000 5850
-F 0 "P25" H 6050 5550 50  0000 C CNN
+F 0 "P25" H 6000 5550 50  0000 C CNN
 F 1 "CONN_4" V 6100 5800 50  0000 C CNN
 F 2 "" H 6000 5850 50  0001 C CNN
@@
 	1    4550 5750
 	0    1    1    0
-$EndComp
-$Comp
-L switches:SW_SPDT_MSM SW14
-U 1 1 4EB6CD1F
-P 7850 1300
-F 0 "SW14" H 7500 1200 50  0000 C CNN
-F 1 "RIGHT_3P1V" H 8900 1250 50  0000 C CNN
-F 2 "" H 7850 1300 50  0001 C CNN
-F 3 "" H 7850 1300 50  0001 C CNN
-	1    7850 1300
-	-1   0    0    -1
 $EndComp
 Text Notes 9700 4900 2    60   ~ 0
@@
 NoConn ~ 8950 5150
 $Comp
-L switches:SW_SPDT_MSM SW15
+L switches:SW_SPDT_MSM SW16
 U 1 1 4EB6CD1D
 P 7850 1700
-F 0 "SW15" H 7500 1600 50  0000 C CNN
+F 0 "SW16" H 7500 1600 50  0000 C CNN
 F 1 "RIGHT_3P1V" H 8900 1700 50  0000 C CNN
 F 2 "" H 7850 1700 50  0001 C CNN
@@
 $EndComp
 $Comp
-L switches:SW_SPDT_MSM SW16
+L switches:SW_SPDT_MSM SW17
 U 1 1 4EB6CD1C
 P 7850 2100
-F 0 "SW16" H 7500 2000 50  0000 C CNN
+F 0 "SW17" H 7500 2000 50  0000 C CNN
 F 1 "RIGHT_3P1V" H 8900 2050 50  0000 C CNN
 F 2 "" H 7850 2100 50  0001 C CNN
@@
 $EndComp
 $Comp
-L switches:SW_SPDT_MSM SW17
+L switches:SW_SPDT_MSM SW18
 U 1 1 4EB6CD1B
 P 7850 2500
-F 0 "SW17" H 7500 2400 50  0000 C CNN
+F 0 "SW18" H 7500 2400 50  0000 C CNN
 F 1 "RIGHT_3P1V" H 8900 2500 50  0000 C CNN
 F 2 "" H 7850 2500 50  0001 C CNN
@@
 $EndComp
 $Comp
-L switches:SW_SPDT_MSM SW18
+L switches:SW_SPDT_MSM SW19
 U 1 1 4EB6CD1A
 P 7850 2900
-F 0 "SW18" H 7500 2800 50  0000 C CNN
+F 0 "SW19" H 7500 2800 50  0000 C CNN
 F 1 "RIGHT_3P1V" H 8900 2900 50  0000 C CNN
 F 2 "" H 7850 2900 50  0001 C CNN
@@
 $EndComp
 $Comp
-L switches:SW_SPDT_MSM SW19
+L switches:SW_SPDT_MSM SW20
 U 1 1 4EB6CD19
 P 7850 3300
-F 0 "SW19" H 7500 3200 50  0000 C CNN
+F 0 "SW20" H 7500 3200 50  0000 C CNN
 F 1 "RIGHT_3P1V" H 8900 3300 50  0000 C CNN
 F 2 "" H 7850 3300 50  0001 C CNN
@@
 $EndComp
 $Comp
-L switches:SW_SPDT_MSM SW20
+L switches:SW_SPDT_MSM SW21
 U 1 1 4EB6CD18
 P 7850 3700
-F 0 "SW20" H 7500 3600 50  0000 C CNN
+F 0 "SW21" H 7500 3600 50  0000 C CNN
 F 1 "RIGHT_3P1V" H 8900 3700 50  0000 C CNN
 F 2 "" H 7850 3700 50  0001 C CNN
@@
 $EndComp
 $Comp
-L switches:SW_SPDT_MSM SW21
+L switches:SW_SPDT_MSM SW22
 U 1 1 4EB6CD17
 P 7850 4100
-F 0 "SW21" H 7500 4000 50  0000 C CNN
+F 0 "SW22" H 7500 4000 50  0000 C CNN
 F 1 "RIGHT_3P1V" H 8900 4100 50  0000 C CNN
 F 2 "" H 7850 4100 50  0001 C CNN
@@
 $EndComp
 $Comp
-L switches:SW_SPDT_MSM SW22
+L switches:SW_SPDT_MSM SW23
 U 1 1 4EB6CD16
 P 7850 4500
-F 0 "SW22" H 7500 4400 50  0000 C CNN
+F 0 "SW23" H 7500 4400 50  0000 C CNN
 F 1 "RIGHT_3P1V" H 8900 4500 50  0000 C CNN
 F 2 "" H 7850 4500 50  0001 C CNN
@@
 	4200 6650 4200 6900
 $Comp
-L switches:SW_SPDT_MSM SW5
-U 1 1 4E47CA5F
-P 2600 1250
-F 0 "SW5" H 2250 1150 50  0000 C CNN
-F 1 "LEFT_3P2V" H 3750 1200 50  0000 C CNN
-F 2 "" H 2600 1250 50  0001 C CNN
-F 3 "" H 2600 1250 50  0001 C CNN
-	1    2600 1250
-	-1   0    0    -1
-$EndComp
-$Comp
 L switches:SW_SPDT_MSM SW6
 U 1 1 4EAF0CE7
@@
 U 1 1 4EB6CBB7
 P 3900 2850
-F 0 "P23" H 3900 2400 60  0000 C CNN
+F 0 "P23" H 3900 2350 60  0000 C CNN
 F 1 "MULTI_DIGITAL_1" V 4000 2850 60  0000 C CNN
 F 2 "" H 3900 2850 50  0001 C CNN
@@
 	1    0    0    -1
 $EndComp
-$Comp
-L switches:SW_SPDT_MSM SW4
-U 1 1 4EB6CDBE
-P 2600 850
-F 0 "SW4" H 2950 650 50  0000 C CNN
-F 1 "RF_SWITCH_3P2V" H 1350 800 50  0000 C CNN
-F 2 "" H 2600 850 50  0001 C CNN
-F 3 "" H 2600 850 50  0001 C CNN
-	1    2600 850
-	1    0    0    -1
-$EndComp
-Wire Notes Line
-	2600 1250 2600 850
 Wire Wire Line
 	2800 2850 3700 2850
@@
 $EndComp
 $Comp
-L conn:Conn_01x03 K1
+L conn:Conn_01x03 P1
 U 1 1 4EB6D0B4
 P 3100 5850
-F 0 "K1" H 3100 5650 50  0000 C CNN
+F 0 "P1" H 3100 5650 50  0000 C CNN
 F 1 "CONN_3" V 3200 5850 40  0000 C CNN
 F 2 "" H 3100 5850 50  0001 C CNN
@@
 	2000 850  2400 850
 $Comp
-L conn:Conn_01x05 P28
+L conn:Conn_01x04 P28
 U 1 1 5DE76C1C
 P 9150 4950
-F 0 "P28" H 9100 5250 50  0000 L CNN
+F 0 "P28" H 9100 4650 50  0000 L CNN
 F 1 "PWR_BUS" V 9250 4750 50  0000 L CNN
 F 2 "" H 9150 4950 50  0001 C CNN
@@
 	1    0    0    -1
 $EndComp
-NoConn ~ 8950 4750
-Text Notes 9750 4800 2    60   ~ 0
-+1.65V
 Text Notes 4450 4850 2    60   ~ 0
 +3.3V
@@
 VBAT+
 $Comp
-L conn:Conn_01x05 P24
+L conn:Conn_01x04 P24
 U 1 1 5DE9BBDD
 P 3900 4900
-F 0 "P24" H 3850 5200 50  0000 L CNN
+F 0 "P24" H 3850 4600 50  0000 L CNN
 F 1 "PWR_BUS" V 4000 4700 50  0000 L CNN
 F 2 "" H 3900 4900 50  0001 C CNN
@@
 	1    0    0    -1
 $EndComp
-Text Notes 4500 4750 2    60   ~ 0
-+1.65V
 Text Notes 3650 6500 2    60   ~ 0
 +3.3V
@@
 VBAT+
 $Comp
-L conn:Conn_01x05 P21
+L conn:Conn_01x04 P21
 U 1 1 5DEA4D3C
 P 3100 6550
-F 0 "P21" H 3050 6850 50  0000 L CNN
+F 0 "P21" H 3050 6250 50  0000 L CNN
 F 1 "PWR_BUS" V 3200 6350 50  0000 L CNN
 F 2 "" H 3100 6550 50  0001 C CNN
@@
 	1    0    0    -1
 $EndComp
-Text Notes 3700 6400 2    60   ~ 0
-+1.65V
 Text Notes 6550 6950 2    60   ~ 0
 +3.3V
@@
 VBAT+
 $Comp
-L conn:Conn_01x05 P26
+L conn:Conn_01x04 P26
 U 1 1 5DEAE08F
 P 6000 7000
-F 0 "P26" H 5950 7300 50  0000 L CNN
+F 0 "P26" H 5950 6700 50  0000 L CNN
 F 1 "PWR_BUS" V 6100 6800 50  0000 L CNN
 F 2 "" H 6000 7000 50  0001 C CNN
@@
 	1    0    0    -1
 $EndComp
-Text Notes 6600 6850 2    60   ~ 0
-+1.65V
-NoConn ~ 5800 6800
-NoConn ~ 2900 6350
-NoConn ~ 3700 4700
-NoConn ~ 1550 5300
 NoConn ~ 3700 5100
+$Comp
+L switches:SW_SP3T SW4
+U 1 1 5D9ED3FC
+P 2600 850
+F 0 "SW4" H 2950 650 50  0000 C CNN
+F 1 "RF_SWITCH_3P2V" H 1350 850 50  0000 C CNN
+F 2 "" H 1975 1025 50  0001 C CNN
+F 3 "" H 1975 1025 50  0001 C CNN
+	1    2600 850
+	1    0    0    -1
+$EndComp
+$Comp
+L switches:SW_SP3T SW5
+U 1 1 5D9EE323
+P 2600 1250
+F 0 "SW5" H 2250 1150 50  0000 C CNN
+F 1 "LEFT_3P2V" H 3750 1250 50  0000 C CNN
+F 2 "" H 1975 1425 50  0001 C CNN
+F 3 "" H 1975 1425 50  0001 C CNN
+	1    2600 1250
+	-1   0    0    -1
+$EndComp
+$Comp
+L switches:SW_SP3T SW15
+U 1 1 5D9EE3BE
+P 7850 1300
+F 0 "SW15" H 7500 1200 50  0000 C CNN
+F 1 "RIGHT_3P2V_A" H 8950 1300 50  0000 C CNN
+F 2 "" H 7225 1475 50  0001 C CNN
+F 3 "" H 7225 1475 50  0001 C CNN
+	1    7850 1300
+	-1   0    0    -1
+$EndComp
+Wire Notes Line
+	2600 1200 2600 800
+NoConn ~ 2400 1250
+NoConn ~ 2800 850
+NoConn ~ 2800 950
+NoConn ~ 7650 1300
+$Comp
+L switches:SW_SP3T SW14
+U 1 1 5DA2B20E
+P 7850 900
+F 0 "SW14" H 7500 800 50  0000 C CNN
+F 1 "RIGHT_3P2V_B" H 8950 900 50  0000 C CNN
+F 2 "" H 7225 1075 50  0001 C CNN
+F 3 "" H 7225 1075 50  0001 C CNN
+	1    7850 900
+	-1   0    0    -1
+$EndComp
+NoConn ~ 8050 900
+NoConn ~ 7650 800
+NoConn ~ 7650 900
+NoConn ~ 7650 1000
+Wire Notes Line
+	7850 850  7850 1250
+Wire Notes Line
+	7600 750  7600 1500
+Wire Notes Line
+	7600 1500 8100 1500
+Wire Notes Line
+	8100 1500 8100 750
+Wire Notes Line
+	8100 750  7600 750
+Wire Notes Line
+	2350 700  2350 1450
+Wire Notes Line
+	2350 1450 2850 1450
+Wire Notes Line
+	2850 1450 2850 700
+Wire Notes Line
+	2850 700  2350 700
+$Comp
+L power:+3.3V #PWR?
+U 1 1 5F85DD3F
+P 7250 1100
+F 0 "#PWR?" H 7250 950 50  0001 C CNN
+F 1 "+3.3V" H 7265 1273 50  0000 C CNN
+F 2 "" H 7250 1100 50  0001 C CNN
+F 3 "" H 7250 1100 50  0001 C CNN
+	1    7250 1100
+	1    0    0    -1
+$EndComp
+$Comp
+L power:+3.3V #PWR?
+U 1 1 5F85F799
+P 4200 5650
+F 0 "#PWR?" H 4200 5500 50  0001 C CNN
+F 1 "+3.3V" H 4215 5823 50  0000 C CNN
+F 2 "" H 4200 5650 50  0001 C CNN
+F 3 "" H 4200 5650 50  0001 C CNN
+	1    4200 5650
+	1    0    0    -1
+$EndComp
+$Comp
+L power:+3.3V #PWR?
+U 1 1 5F86063A
+P 2000 1100
+F 0 "#PWR?" H 2000 950 50  0001 C CNN
+F 1 "+3.3V" H 2015 1273 50  0000 C CNN
+F 2 "" H 2000 1100 50  0001 C CNN
+F 3 "" H 2000 1100 50  0001 C CNN
+	1    2000 1100
+	1    0    0    -1
+$EndComp
+$Comp
+L power:GND #PWR?
+U 1 1 5F861623
+P 7150 5150
+F 0 "#PWR?" H 7150 4900 50  0001 C CNN
+F 1 "GND" H 7155 4977 50  0000 C CNN
+F 2 "" H 7150 5150 50  0001 C CNN
+F 3 "" H 7150 5150 50  0001 C CNN
+	1    7150 5150
+	1    0    0    -1
+$EndComp
+$Comp
+L power:GND #PWR?
+U 1 1 5F862221
+P 4200 7000
+F 0 "#PWR?" H 4200 6750 50  0001 C CNN
+F 1 "GND" H 4205 6827 50  0000 C CNN
+F 2 "" H 4200 7000 50  0001 C CNN
+F 3 "" H 4200 7000 50  0001 C CNN
+	1    4200 7000
+	1    0    0    -1
+$EndComp
+$Comp
+L power:GND #PWR?
+U 1 1 5F863347
+P 1250 6750
+F 0 "#PWR?" H 1250 6500 50  0001 C CNN
+F 1 "GND" H 1255 6577 50  0000 C CNN
+F 2 "" H 1250 6750 50  0001 C CNN
+F 3 "" H 1250 6750 50  0001 C CNN
+	1    1250 6750
+	1    0    0    -1
+$EndComp
+$Comp
+L power:GND #PWR?
+U 1 1 5F864106
+P 1900 5100
+F 0 "#PWR?" H 1900 4850 50  0001 C CNN
+F 1 "GND" H 1905 4927 50  0000 C CNN
+F 2 "" H 1900 5100 50  0001 C CNN
+F 3 "" H 1900 5100 50  0001 C CNN
+	1    1900 5100
+	1    0    0    -1
+$EndComp
+Wire Wire Line
+	7250 1100 7250 1200
+Connection ~ 7250 1200
+Wire Wire Line
+	7150 5050 7150 5150
+Connection ~ 7150 5050
+Wire Wire Line
+	4200 6900 4200 7000
+Connection ~ 4200 6900
+Wire Wire Line
+	1250 6650 1250 6750
+Connection ~ 1250 6650
+Wire Wire Line
+	1900 5000 1900 5100
+Connection ~ 1900 5000
+Wire Wire Line
+	2000 1100 2000 1150
+Connection ~ 2000 1150
+Wire Wire Line
+	4200 5650 4200 5750
+Connection ~ 4200 5750
 $EndSCHEMATC

Commit message: Adding footprints
Parts:
- D2, D3, D4, D5: footprint (none) -> LEDs:LED_D3.0mm; symbol device:LED -> RCTX-rescue:LED-device
- P22: renamed from P1; value CONN_3 -> SW; footprint (none) -> Connectors_Samtec:SL-103-X-XX_1x03; symbol conn:Conn_01x03 -> RCTX-rescue:Conn_01x03-conn
- P23: renamed from P21; footprint (none) -> Connectors_Samtec:SL-104-X-XX_1x04; symbol conn:Conn_01x04 -> RCTX-rescue:Conn_01x04-conn
- P24: renamed from P22; footprint (none) -> Connectors_Samtec:SL-102-X-XX_1x02; symbol conn:Conn_01x02 -> RCTX-rescue:Conn_01x02-conn
- P25: renamed from P23; footprint (none) -> Connectors_Samtec:SL-109-X-XX_1x09; symbol conn:Conn_01x09 -> RCTX-rescue:Conn_01x09-conn
- P26: renamed from P24; footprint (none) -> Connectors_Samtec:SL-104-X-XX_1x04; symbol conn:Conn_01x04 -> RCTX-rescue:Conn_01x04-conn
- P27: renamed from P25; value CONN_4 -> LEDS; footprint (none) -> Connectors_Samtec:SL-104-X-XX_1x04; symbol conn:Conn_01x04 -> RCTX-rescue:Conn_01x04-conn
- P28: renamed from P26; footprint (none) -> Connectors_Samtec:SL-104-X-XX_1x04; symbol conn:Conn_01x04 -> RCTX-rescue:Conn_01x04-conn
- P29: renamed from P27; footprint (none) -> Connectors_Samtec:SL-109-X-XX_1x09; symbol conn:Conn_01x09 -> RCTX-rescue:Conn_01x09-conn
- P30: renamed from P28; footprint (none) -> Connectors_Samtec:SL-104-X-XX_1x04; symbol conn:Conn_01x04 -> RCTX-rescue:Conn_01x04-conn
- R5: renamed from R4; footprint (none) -> Resistors_THT:R_Axial_DIN0204_L3.6mm_D1.6mm_P1.90mm_Vertical; symbol device:R -> RCTX-rescue:R-device
- R6: renamed from R5; footprint (none) -> Resistors_THT:R_Axial_DIN0204_L3.6mm_D1.6mm_P1.90mm_Vertical; symbol device:R -> RCTX-rescue:R-device
- R7: renamed from R6; footprint (none) -> Resistors_THT:R_Axial_DIN0204_L3.6mm_D1.6mm_P1.90mm_Vertical; symbol device:R -> RCTX-rescue:R-device
- R8: renamed from R7; footprint (none) -> Resistors_THT:R_Axial_DIN0204_L3.6mm_D1.6mm_P1.90mm_Vertical; symbol device:R -> RCTX-rescue:R-device
- SW1, SW2, SW3: footprint (none) -> Buttons_Switches_THT:SW_PUSH_6mm_h5mm; symbol switches:SW_SPST -> RCTX-rescue:SW_SPST-switches
- SW10, SW11, SW12, SW13, SW16, SW17, SW18, SW19, SW20, SW21, SW22, SW23, SW6, SW7, SW8, SW9: footprint (none) -> Buttons_Switches_THT:SW_CuK_JS202011CQN_DPDT_Straight; symbol switches:SW_SPDT_MSM -> RCTX-rescue:SW_SPDT_MSM-switches
- SW14, SW15, SW4, SW5: footprint (none) -> Buttons_Switches_THT:SW_CuK_JS202011AQN_DPDT_Angled; symbol switches:SW_SP3T -> RCTX-rescue:SW_SP3T-switches
