File: kicad/RCTX_MDL.sch (KiCad schematic (older format))
At the start: 40 parts, among them P22 SW, P23 PWR_BUS, P24 TX_VCC, P25 MULTI_DIGITAL_1, P26 PWR_BUS, P27 LEDS, P28 PWR_BUS, P29 MULTI_DIGITAL_2, P30 PWR_BUS, SW1 Reset, SW10 LEFT_3P1V, SW11 LEFT_3P1V, SW12 LEFT_3P1V, SW13 LEFT_3P1V, SW14 RIGHT_3P2V_B, SW15 RIGHT_3P2V_A, SW16 RIGHT_3P1V, SW17 RIGHT_3P1V, SW18 RIGHT_3P1V, SW19 RIGHT_3P1V, SW2 Program, SW20 RIGHT_3P1V, SW21 RIGHT_3P1V, SW22 RIGHT_3P1V, SW23 RIGHT_3P1V, SW3 User, SW4 RF_SWITCH_3P2V, SW5 LEFT_3P2V, SW6 LEFT_3P1V, SW7 LEFT_3P1V, SW8 LEFT_3P1V, SW9 LEFT_3P1V

Commit message: Fixing keypad wiring
Parts:
- renumbered SW6 to SW1, SW17 to SW10, SW18 to SW11, SW19 to SW12, SW20 to SW13, SW21 to SW14, SW22 to SW15, SW23 to SW16, SW4 to SW17, SW5 to SW18, SW14 to SW19, SW7 to SW2, SW15 to SW20, SW8 to SW3, SW9 to SW4, SW10 to SW5, SW11 to SW6, SW12 to SW7, SW13 to SW8, SW16 to SW9
Changed lines of the file:
@@
 NoConn ~ 8950 5150
 $Comp
-L RCTX-rescue:SW_SPDT_MSM-switches SW16
+L RCTX-rescue:SW_SPDT_MSM-switches SW9
 U 1 1 4EB6CD1D
 P 7850 1700
-F 0 "SW16" H 7500 1600 50  0000 C CNN
+F 0 "SW9" H 7450 1600 50  0000 C CNN
 F 1 "RIGHT_3P1V" H 8900 1700 50  0000 C CNN
 F 2 "Buttons_Switches_THT:SW_CuK_JS202011CQN_DPDT_Straight" H 7850 1700 50  0001 C CNN
@@
 $EndComp
 $Comp
-L RCTX-rescue:SW_SPDT_MSM-switches SW17
+L RCTX-rescue:SW_SPDT_MSM-switches SW10
 U 1 1 4EB6CD1C
 P 7850 2100
-F 0 "SW17" H 7500 2000 50  0000 C CNN
+F 0 "SW10" H 7450 2000 50  0000 C CNN
 F 1 "RIGHT_3P1V" H 8900 2050 50  0000 C CNN
 F 2 "Buttons_Switches_THT:SW_CuK_JS202011CQN_DPDT_Straight" H 7850 2100 50  0001 C CNN
@@
 $EndComp
 $Comp
-L RCTX-rescue:SW_SPDT_MSM-switches SW18
+L RCTX-rescue:SW_SPDT_MSM-switches SW11
 U 1 1 4EB6CD1B
 P 7850 2500
-F 0 "SW18" H 7500 2400 50  0000 C CNN
+F 0 "SW11" H 7450 2400 50  0000 C CNN
 F 1 "RIGHT_3P1V" H 8900 2500 50  0000 C CNN
 F 2 "Buttons_Switches_THT:SW_CuK_JS202011CQN_DPDT_Straight" H 7850 2500 50  0001 C CNN
@@
 $EndComp
 $Comp
-L RCTX-rescue:SW_SPDT_MSM-switches SW19
+L RCTX-rescue:SW_SPDT_MSM-switches SW12
 U 1 1 4EB6CD1A
 P 7850 2900
-F 0 "SW19" H 7500 2800 50  0000 C CNN
+F 0 "SW12" H 7450 2800 50  0000 C CNN
 F 1 "RIGHT_3P1V" H 8900 2900 50  0000 C CNN
 F 2 "Buttons_Switches_THT:SW_CuK_JS202011CQN_DPDT_Straight" H 7850 2900 50  0001 C CNN
@@
 $EndComp
 $Comp
-L RCTX-rescue:SW_SPDT_MSM-switches SW20
+L RCTX-rescue:SW_SPDT_MSM-switches SW13
 U 1 1 4EB6CD19
 P 7850 3300
-F 0 "SW20" H 7500 3200 50  0000 C CNN
+F 0 "SW13" H 7450 3200 50  0000 C CNN
 F 1 "RIGHT_3P1V" H 8900 3300 50  0000 C CNN
 F 2 "Buttons_Switches_THT:SW_CuK_JS202011CQN_DPDT_Straight" H 7850 3300 50  0001 C CNN
@@
 $EndComp
 $Comp
-L RCTX-rescue:SW_SPDT_MSM-switches SW21
+L RCTX-rescue:SW_SPDT_MSM-switches SW14
 U 1 1 4EB6CD18
 P 7850 3700
-F 0 "SW21" H 7500 3600 50  0000 C CNN
+F 0 "SW14" H 7450 3600 50  0000 C CNN
 F 1 "RIGHT_3P1V" H 8900 3700 50  0000 C CNN
 F 2 "Buttons_Switches_THT:SW_CuK_JS202011CQN_DPDT_Straight" H 7850 3700 50  0001 C CNN
@@
 $EndComp
 $Comp
-L RCTX-rescue:SW_SPDT_MSM-switches SW22
+L RCTX-rescue:SW_SPDT_MSM-switches SW15
 U 1 1 4EB6CD17
 P 7850 4100
-F 0 "SW22" H 7500 4000 50  0000 C CNN
+F 0 "SW15" H 7450 4000 50  0000 C CNN
 F 1 "RIGHT_3P1V" H 8900 4100 50  0000 C CNN
 F 2 "Buttons_Switches_THT:SW_CuK_JS202011CQN_DPDT_Straight" H 7850 4100 50  0001 C CNN
@@
 $EndComp
 $Comp
-L RCTX-rescue:SW_SPDT_MSM-switches SW23
+L RCTX-rescue:SW_SPDT_MSM-switches SW16
 U 1 1 4EB6CD16
 P 7850 4500
-F 0 "SW23" H 7500 4400 50  0000 C CNN
+F 0 "SW16" H 7450 4400 50  0000 C CNN
 F 1 "RIGHT_3P1V" H 8900 4500 50  0000 C CNN
 F 2 "Buttons_Switches_THT:SW_CuK_JS202011CQN_DPDT_Straight" H 7850 4500 50  0001 C CNN
@@
 	4200 6650 4200 6900
 $Comp
-L RCTX-rescue:SW_SPDT_MSM-switches SW6
+L RCTX-rescue:SW_SPDT_MSM-switches SW1
 U 1 1 4EAF0CE7
 P 2600 1650
-F 0 "SW6" H 2250 1550 50  0000 C CNN
+F 0 "SW1" H 2200 1550 50  0000 C CNN
 F 1 "LEFT_3P1V" H 3750 1650 50  0000 C CNN
 F 2 "Buttons_Switches_THT:SW_CuK_JS202011CQN_DPDT_Straight" H 2600 1650 50  0001 C CNN
@@
 $EndComp
 $Comp
-L RCTX-rescue:SW_SPDT_MSM-switches SW7
+L RCTX-rescue:SW_SPDT_MSM-switches SW2
 U 1 1 4EAF0CEA
 P 2600 2050
-F 0 "SW7" H 2250 1950 50  0000 C CNN
+F 0 "SW2" H 2200 1950 50  0000 C CNN
 F 1 "LEFT_3P1V" H 3750 2000 50  0000 C CNN
 F 2 "Buttons_Switches_THT:SW_CuK_JS202011CQN_DPDT_Straight" H 2600 2050 50  0001 C CNN
@@
 $EndComp
 $Comp
-L RCTX-rescue:SW_SPDT_MSM-switches SW8
+L RCTX-rescue:SW_SPDT_MSM-switches SW3
 U 1 1 4EAF0CEC
 P 2600 2450
-F 0 "SW8" H 2250 2350 50  0000 C CNN
+F 0 "SW3" H 2200 2350 50  0000 C CNN
 F 1 "LEFT_3P1V" H 3750 2400 50  0000 C CNN
 F 2 "Buttons_Switches_THT:SW_CuK_JS202011CQN_DPDT_Straight" H 2600 2450 50  0001 C CNN
@@
 $EndComp
 $Comp
-L RCTX-rescue:SW_SPDT_MSM-switches SW9
+L RCTX-rescue:SW_SPDT_MSM-switches SW4
 U 1 1 4EAF0CEE
 P 2600 2850
-F 0 "SW9" H 2250 2750 50  0000 C CNN
+F 0 "SW4" H 2200 2750 50  0000 C CNN
 F 1 "LEFT_3P1V" H 3750 2850 50  0000 C CNN
 F 2 "Buttons_Switches_THT:SW_CuK_JS202011CQN_DPDT_Straight" H 2600 2850 50  0001 C CNN
@@
 $EndComp
 $Comp
-L RCTX-rescue:SW_SPDT_MSM-switches SW10
+L RCTX-rescue:SW_SPDT_MSM-switches SW5
 U 1 1 4EAF0CF0
 P 2600 3250
-F 0 "SW10" H 2250 3150 50  0000 C CNN
+F 0 "SW5" H 2200 3150 50  0000 C CNN
 F 1 "LEFT_3P1V" H 3750 3200 50  0000 C CNN
 F 2 "Buttons_Switches_THT:SW_CuK_JS202011CQN_DPDT_Straight" H 2600 3250 50  0001 C CNN
@@
 $EndComp
 $Comp
-L RCTX-rescue:SW_SPDT_MSM-switches SW11
+L RCTX-rescue:SW_SPDT_MSM-switches SW6
 U 1 1 4EAF0CF3
 P 2600 3650
-F 0 "SW11" H 2250 3550 50  0000 C CNN
+F 0 "SW6" H 2200 3550 50  0000 C CNN
 F 1 "LEFT_3P1V" H 3750 3650 50  0000 C CNN
 F 2 "Buttons_Switches_THT:SW_CuK_JS202011CQN_DPDT_Straight" H 2600 3650 50  0001 C CNN
@@
 $EndComp
 $Comp
-L RCTX-rescue:SW_SPDT_MSM-switches SW12
+L RCTX-rescue:SW_SPDT_MSM-switches SW7
 U 1 1 4EAF0CF6
 P 2600 4050
-F 0 "SW12" H 2250 3950 50  0000 C CNN
+F 0 "SW7" H 2200 3950 50  0000 C CNN
 F 1 "LEFT_3P1V" H 3750 4000 50  0000 C CNN
 F 2 "Buttons_Switches_THT:SW_CuK_JS202011CQN_DPDT_Straight" H 2600 4050 50  0001 C CNN
@@
 $EndComp
 $Comp
-L RCTX-rescue:SW_SPDT_MSM-switches SW13
+L RCTX-rescue:SW_SPDT_MSM-switches SW8
 U 1 1 4EAF0CF8
 P 2600 4450
-F 0 "SW13" H 2250 4350 50  0000 C CNN
+F 0 "SW8" H 2200 4350 50  0000 C CNN
 F 1 "LEFT_3P1V" H 3750 4450 50  0000 C CNN
 F 2 "Buttons_Switches_THT:SW_CuK_JS202011CQN_DPDT_Straight" H 2600 4450 50  0001 C CNN
@@
 NoConn ~ 3700 5100
 $Comp
-L RCTX-rescue:SW_SP3T-switches SW4
+L RCTX-rescue:SW_SP3T-switches SW17
 U 1 1 5D9ED3FC
 P 2600 850
-F 0 "SW4" H 2950 650 50  0000 C CNN
+F 0 "SW17" H 3000 650 50  0000 C CNN
 F 1 "RF_SWITCH_3P2V" H 1350 850 50  0000 C CNN
 F 2 "Buttons_Switches_THT:SW_CuK_JS202011AQN_DPDT_Angled" H 1975 1025 50  0001 C CNN
@@
 $EndComp
 $Comp
-L RCTX-rescue:SW_SP3T-switches SW5
+L RCTX-rescue:SW_SP3T-switches SW18
 U 1 1 5D9EE323
 P 2600 1250
-F 0 "SW5" H 2250 1150 50  0000 C CNN
+F 0 "SW18" H 2200 1150 50  0000 C CNN
 F 1 "LEFT_3P2V" H 3750 1250 50  0000 C CNN
 F 2 "Buttons_Switches_THT:SW_CuK_JS202011AQN_DPDT_Angled" H 1975 1425 50  0001 C CNN
@@
 $EndComp
 $Comp
-L RCTX-rescue:SW_SP3T-switches SW15
+L RCTX-rescue:SW_SP3T-switches SW20
 U 1 1 5D9EE3BE
 P 7850 1300
-F 0 "SW15" H 7500 1200 50  0000 C CNN
+F 0 "SW20" H 7450 1200 50  0000 C CNN
 F 1 "RIGHT_3P2V_A" H 8950 1300 50  0000 C CNN
 F 2 "Buttons_Switches_THT:SW_CuK_JS202011AQN_DPDT_Angled" H 7225 1475 50  0001 C CNN
@@
 NoConn ~ 7650 1300
 $Comp
-L RCTX-rescue:SW_SP3T-switches SW14
+L RCTX-rescue:SW_SP3T-switches SW19
 U 1 1 5DA2B20E
 P 7850 900
-F 0 "SW14" H 7500 800 50  0000 C CNN
+F 0 "SW19" H 7450 800 50  0000 C CNN
 F 1 "RIGHT_3P2V_B" H 8950 900 50  0000 C CNN
 F 2 "Buttons_Switches_THT:SW_CuK_JS202011AQN_DPDT_Angled" H 7225 1075 50  0001 C CNN
