File: kicad/RCTX_MP.sch (KiCad schematic (older format))
At the start: 22 parts, among them J24 ROTARY_4, J25 ROTARY_5, J26 ROTARY_3, J27 ROTARY_6, J28 ROTARY_2, J29 ROTARY_7, J30 ROTARY_1, J31 ROTARY_8, J32 PWR_BUS, J33 H_RIGHT_JOYSTIC, J34 ROTARY_9, J35 V_RIGHT_JOYSTIC, J36 ROTARY_10, J37 H_LEFT_JOYSTIC, J38 ROTARY_11, J39 V_LEFT_JOYSTIC, J40 ROTARY_12, J41 MULTI_PROP_1, J42 MULTI_PROP_2, U9 LM324

Commit message: Adding 5110 display
Parts:
- added C?: 1uF, symbol device:CP
- added C?: 100nF, symbol device:C
- added R?: 470, symbol device:R
- added R?: 150, symbol device:R
- added U?: LM117_TO3, TO_SOT_Packages_THT:TO-3, symbol regul:LM117_TO3
- J32: symbol conn:Conn_01x05 -> conn:Conn_01x04
Connections:
- net GND: now reaches C16.1, C17.2, J24.1 (Pin_1), J25.1 (Pin_1), J26.1 (Pin_1), J27.1 (Pin_1), J28.1 (Pin_1), J29.1 (Pin_1), J30.1 (Pin_1), J31.1 (Pin_1), J33.1 (Pin_1), J34.1 (Pin_1), J35.1 (Pin_1), J36.1 (Pin_1), J37.1 (Pin_1), J38.1 (Pin_1), J39.1 (Pin_1), J40.1 (Pin_1), U9.11 (V-), U9.11 (V-), U9.11 (V-), U9.11 (V-)
- net GND: now also J32.3 (Pin_3), C?.2, C?.2, R?.1; no longer J32.4 (Pin_4)
- net at J24.3 (Pin_3), J25.3 (Pin_3), J26.3 (Pin_3)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: now also C?.1, R?.1, U?.3 (VO); no longer J32.1 (Pin_1)
- net +5V: now reaches C16.2, C17.1, U9.4 (V+), U9.4 (V+), U9.4 (V+), U9.4 (V+)
- net +5V: now also J32.2 (Pin_2); no longer J32.3 (Pin_3)
- net +3V3: now reaches J33.3 (Pin_3), J35.3 (Pin_3), J37.3 (Pin_3), J39.3 (Pin_3)
- net +3V3: now also J32.1 (Pin_1), C?.1, U?.2 (VI); no longer J32.2 (Pin_2)
- new net: R?.2, R?.2, U?.1 (ADJ)
Other:
- note removed: "+1.65V"
- moved on the sheet: C16, C17, J24, J25, J26, J27, J28, J29, J30, J31, J33, J34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

Commit message: Adding footprints
Parts:
- C17: renamed from C?; footprint (none) -> Capacitors_THT:CP_Radial_D5.0mm_P2.50mm; symbol device:CP -> RCTX-rescue:CP-device
- C18: renamed from C?; footprint (none) -> Capacitors_THT:C_Disc_D3.0mm_W1.6mm_P2.50mm; symbol device:C -> RCTX-rescue:C-device
- C19: renamed from C16; footprint (none) -> Capacitors_THT:C_Disc_D3.0mm_W1.6mm_P2.50mm; symbol device:C -> RCTX-rescue:C-device
- C20: renamed from C17; footprint (none) -> Capacitors_THT:CP_Radial_D5.0mm_P2.50mm; symbol device:CP -> RCTX-rescue:CP-device
- J24, J25, J26, J27, J28, J29, J30, J31, J33, J34, J35, J36, J37, J38, J39, J40: footprint (none) -> servo_conn:SRV_1; symbol conn:Conn_01x03 -> RCTX-rescue:Conn_01x03-conn
- J32: footprint (none) -> Connectors_Samtec:SL-104-X-XX_1x04; symbol conn:Conn_01x04 -> RCTX-rescue:Conn_01x04-conn
- J41, J42: footprint (none) -> Connectors_Samtec:SL-108-X-XX_1x08; symbol conn:Conn_01x08 -> RCTX-rescue:Conn_01x08-conn
- R11, R12: renamed from R?; footprint (none) -> Resistors_THT:R_Axial_DIN0204_L3.6mm_D1.6mm_P1.90mm_Vertical; symbol device:R -> RCTX-rescue:R-device
- U10: renamed from U?; footprint TO_SOT_Packages_THT:TO-3 -> TO_SOT_Packages_THT:TO-92_Inline_Narrow_Oval; symbol regul:LM117_TO3 -> RCTX-rescue:LM117_TO3-regul
- U11: renamed from U9; footprint (none) -> Housings_DIP:DIP-14_W7.62mm; symbol linear:LM324 -> RCTX-rescue:LM324-linear
