File: kicad/RCTX_MP.sch (KiCad schematic (older format))
At the start: 27 parts, among them J24 ROTARY_4, J25 ROTARY_5, J26 ROTARY_3, J27 ROTARY_6, J28 ROTARY_2, J29 ROTARY_7, J30 ROTARY_1, J31 ROTARY_8, J32 PWR_BUS, J33 H_RIGHT_JOYSTIC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

Commit message: renaming switches, buttons and trims
Other:
- note added: "ROTARY_01"
- note added: "ROTARY_02"
- note added: "ROTARY_03"
- note added: "ROTARY_04"
- note added: "ROTARY_05"
- note added: "ROTARY_06"
- note added: "ROTARY_07"
- note added: "ROTARY_08"
- note added: "ROTARY_09"
- note added: "ROTARY_10"
- note added: "ROTARY_11"
- note added: "ROTARY_12"
- note removed: "TRIM_1"
- note removed: "TRIM_10"
- note removed: "TRIM_11"
- note removed: "TRIM_12"
- note removed: "TRIM_2"
- note removed: "TRIM_3"
- note removed: "TRIM_4"
- note removed: "TRIM_5"
- note removed: "TRIM_6"
- note removed: "TRIM_7"
- note removed: "TRIM_8"
- note removed: "TRIM_9"
Changed lines of the file:
@@
 NoConn ~ 5000 1300
 Text Notes 10400 2250 1    50   ~ 0
-TRIM_1
+ROTARY_01
 Text Notes 10500 2250 1    50   ~ 0
-TRIM_2
+ROTARY_02
 Text Notes 10600 2250 1    50   ~ 0
-TRIM_3
+ROTARY_03
 Text Notes 10700 2250 1    50   ~ 0
-TRIM_4
-Text Notes 10000 5100 1    50   ~ 0
-TRIM_5
-Text Notes 10100 5100 1    50   ~ 0
-TRIM_6
-Text Notes 10200 5100 1    50   ~ 0
-TRIM_7
-Text Notes 10300 5100 1    50   ~ 0
-TRIM_8
-Text Notes 10400 5100 1    50   ~ 0
-TRIM_9
-Text Notes 10500 5100 1    50   ~ 0
-TRIM_10
-Text Notes 10600 5100 1    50   ~ 0
-TRIM_11
-Text Notes 10700 5100 1    50   ~ 0
-TRIM_12
+ROTARY_04
+Text Notes 10000 5200 1    50   ~ 0
+ROTARY_05
+Text Notes 10100 5200 1    50   ~ 0
+ROTARY_06
+Text Notes 10200 5200 1    50   ~ 0
+ROTARY_07
+Text Notes 10300 5200 1    50   ~ 0
+ROTARY_08
+Text Notes 10400 5200 1    50   ~ 0
+ROTARY_09
+Text Notes 10500 5200 1    50   ~ 0
+ROTARY_10
+Text Notes 10600 5200 1    50   ~ 0
+ROTARY_11
+Text Notes 10700 5200 1    50   ~ 0
+ROTARY_12
 Wire Wire Line
 	3000 1500 4000 1500
