File: kicad/RCTX_TXM.sch (KiCad schematic (older format))
At the start: 17 parts, among them P17 RF MODULE, P18 TX_MOD, P19 PWR_BUS, P20 TX_VCC, Q1 BC547, U1 LM78L05_TO92, U2 MB504L

Commit message: Adding 5110 display
Parts:
- P19: symbol conn:Conn_01x05 -> conn:Conn_01x04
Connections:
- net GND: now reaches AE1.2 (Shield), C2.1, C3.2, C4.2, P17.2 (Pin_2), Q1.3 (E), R2.2, U1.2 (GND), U2.4 (OUT)
- net GND: now also P19.3 (Pin_3); no longer P19.4 (Pin_4)
- net at P17.4 (Pin_4), P20.2 (Pin_2): now also C4.1, U1.3 (VI)
- net +5V: now reaches C2.2, C3.1, U1.1 (VO), U2.2 (VCC), U2.3 (SW), U2.6 (MC)
- net +3V3: now reaches L2.1
- net +3V3: now also P19.1 (Pin_1); no longer P19.3 (Pin_3)
- new net: P19.4 (Pin_4), P20.1 (Pin_1)
- no-connect marks 2 -> 1
Other:
- note added: "/RF_DETECT"
- note added: "FRQ_METER"
- note added: "PPM_OUT"
- note removed: "+1.65V"
- note removed: "FRQ"
- moved on the sheet: P18
Changed lines of the file:
@@
 	4400 4050 4000 4050
 Wire Wire Line
-	5900 2250 6500 2250
+	5900 2150 6500 2150
 Wire Wire Line
-	5900 2250 5900 2700
+	5900 2150 5900 2700
 Wire Wire Line
-	6500 2800 6500 2250
+	6500 2800 6500 2150
 Wire Wire Line
 	5900 4050 7350 4050
 Connection ~ 5900 4050
-Wire Wire Line
-	4800 4550 6500 4550
-Wire Wire Line
-	6500 4550 6500 4150
-Connection ~ 4800 4550
-Wire Wire Line
-	7350 3950 6500 3950
-Wire Wire Line
-	6500 3950 6500 3650
 Text Notes 7750 2300 0    60   ~ 0
-FRQ
+FRQ_METER
 Text Notes 7750 2200 0    60   ~ 0
-LED
+/RF_DETECT
 Text Notes 7750 2100 0    60   ~ 0
-SIG
+PPM_OUT
 $Comp
 L conn:Conn_01x03 P18
 U 1 1 4E4833D2
-P 7550 2150
-F 0 "P18" H 7550 1950 50  0000 C CNN
-F 1 "TX_MOD" V 7650 2150 40  0000 C CNN
-F 2 "" H 7550 2150 50  0001 C CNN
-F 3 "" H 7550 2150 50  0001 C CNN
-	1    7550 2150
+P 7550 2050
+F 0 "P18" H 7550 1850 50  0000 C CNN
+F 1 "TX_MOD" V 7650 2050 40  0000 C CNN
+F 2 "" H 7550 2050 50  0001 C CNN
+F 3 "" H 7550 2050 50  0001 C CNN
+	1    7550 2050
 	1    0    0    1
 $EndComp
 Wire Wire Line
-	6500 2250 7350 2250
-Connection ~ 6500 2250
+	6500 2150 7350 2150
+Connection ~ 6500 2150
 Wire Wire Line
-	2600 2050 7350 2050
+	2600 1950 7350 1950
 Wire Wire Line
-	2700 2150 7350 2150
+	2700 2050 7350 2050
 Wire Wire Line
 	7350 4950 6500 4950
 Wire Wire Line
-	6500 4950 6500 4550
-Wire Wire Line
 	6500 4150 7350 4150
-Connection ~ 6500 4550
 Wire Wire Line
 	2350 3450 2700 3450
 Wire Wire Line
-	2700 3450 2700 2150
+	2700 3450 2700 2050
 Wire Wire Line
 	2350 3650 2600 3650
 Wire Wire Line
-	2600 3650 2600 2050
+	2600 3650 2600 1950
 Wire Wire Line
 	2350 3550 2700 3550
@@
 	2700 3550 2700 5050
 Wire Wire Line
-	2700 5050 7350 5050
+	2700 5050 4800 5050
 Connection ~ 3550 2750
 Connection ~ 3550 3250
@@
 	3150 3200 3150 2800
 $Comp
-L conn:Conn_01x05 P19
+L conn:Conn_01x04 P19
 U 1 1 5DE4A168
 P 7550 3950
@@
 	1    0    0    -1
 $EndComp
-Text Notes 7750 3800 0    60   ~ 0
-+1.65V
-NoConn ~ 7350 3850
-NoConn ~ 7350 3750
+Wire Wire Line
+	6500 4150 6500 4950
+Wire Wire Line
+	4800 4550 4800 5050
+Connection ~ 4800 4550
+Connection ~ 4800 5050
+Wire Wire Line
+	4800 5050 7350 5050
+Wire Wire Line
+	7350 3850 7050 3850
+Wire Wire Line
+	6500 3850 6500 3650
+NoConn ~ 7350 3950
+$Comp
+L power:+3.3V #PWR?
+U 1 1 5F84CE9B
+P 7050 3750
+F 0 "#PWR?" H 7050 3600 50  0001 C CNN
+F 1 "+3.3V" H 7065 3923 50  0000 C CNN
+F 2 "" H 7050 3750 50  0001 C CNN
+F 3 "" H 7050 3750 50  0001 C CNN
+	1    7050 3750
+	1    0    0    -1
+$EndComp
+$Comp
+L power:GND #PWR?
+U 1 1 5F84D89D
+P 5900 4150
+F 0 "#PWR?" H 5900 3900 50  0001 C CNN
+F 1 "GND" H 5905 3977 50  0000 C CNN
+F 2 "" H 5900 4150 50  0001 C CNN
+F 3 "" H 5900 4150 50  0001 C CNN
+	1    5900 4150
+	1    0    0    -1
+$EndComp
+Wire Wire Line
+	7050 3750 7050 3850
+Connection ~ 7050 3850
+Wire Wire Line
+	7050 3850 6500 3850
+Wire Wire Line
+	5900 4150 5900 4050
+$Comp
+L power:+5V #PWR?
+U 1 1 5F8530E2
+P 4450 2350
+F 0 "#PWR?" H 4450 2200 50  0001 C CNN
+F 1 "+5V" H 4465 2523 50  0000 C CNN
+F 2 "" H 4450 2350 50  0001 C CNN
+F 3 "" H 4450 2350 50  0001 C CNN
+	1    4450 2350
+	1    0    0    -1
+$EndComp
+Wire Wire Line
+	4450 2350 4450 2450
 $EndSCHEMATC

Commit message: Adding footprints
Parts:
- AE1: footprint (none) -> Connectors_Samtec:SL-102-X-XX_1x02; symbol device:Antenna_Shield -> RCTX-rescue:Antenna_Shield-device
- C1: renamed from C2; footprint (none) -> Capacitors_THT:C_Disc_D3.0mm_W1.6mm_P2.50mm; symbol device:C -> RCTX-rescue:C-device
- C2: renamed from C3; footprint (none) -> Capacitors_THT:C_Disc_D3.0mm_W1.6mm_P2.50mm; symbol device:C -> RCTX-rescue:C-device
- C3: renamed from C4; footprint (none) -> Capacitors_THT:C_Disc_D3.0mm_W1.6mm_P2.50mm; symbol device:C -> RCTX-rescue:C-device
- C4: renamed from C5; footprint (none) -> Capacitors_THT:C_Disc_D3.0mm_W1.6mm_P2.50mm; symbol device:C -> RCTX-rescue:C-device
- D1: symbol diode:BAV99 -> RCTX-rescue:BAV99-diode
- L1, L2: footprint (none) -> Inductors_THT:L_Axial_L5.3mm_D2.2mm_P2.54mm_Vertical_Vishay_IM-1; symbol device:L -> RCTX-rescue:L-device
- P18: renamed from P17; footprint (none) -> Connectors_Samtec:SL-105-X-XX_1x05; symbol conn:Conn_01x05 -> RCTX-rescue:Conn_01x05-conn
- P19: renamed from P18; footprint (none) -> Connectors_Samtec:SL-103-X-XX_1x03; symbol conn:Conn_01x03 -> RCTX-rescue:Conn_01x03-conn
- P20: renamed from P19; footprint (none) -> Connectors_Samtec:SL-104-X-XX_1x04; symbol conn:Conn_01x04 -> RCTX-rescue:Conn_01x04-conn
- P21: renamed from P20; footprint (none) -> Connectors_Samtec:SL-102-X-XX_1x02; symbol conn:Conn_01x02 -> RCTX-rescue:Conn_01x02-conn
- Q1: symbol transistors:BC547 -> RCTX-rescue:BC547-transistors
- R1: renamed from R2; footprint (none) -> Resistors_THT:R_Axial_DIN0204_L3.6mm_D1.6mm_P1.90mm_Vertical; symbol device:R -> RCTX-rescue:R-device
- R2: renamed from R3; footprint (none) -> Resistors_THT:R_Axial_DIN0204_L3.6mm_D1.6mm_P1.90mm_Vertical; symbol device:R -> RCTX-rescue:R-device
- U1: symbol regul:LM78L05_TO92 -> RCTX-rescue:LM78L05_TO92-regul
- U2: footprint (none) -> Housings_DIP:DIP-8_W7.62mm
Changed lines of the file:
@@
 SIG
 $Comp
-L conn:Conn_01x05 P17
+L RCTX-rescue:Conn_01x05-conn P18
 U 1 1 4DAA052E
 P 2150 3450
-F 0 "P17" H 2150 3150 50  0000 C CNN
+F 0 "P18" H 2150 3150 50  0000 C CNN
 F 1 "RF MODULE" V 2250 3450 50  0000 C CNN
-F 2 "" H 2150 3450 50  0001 C CNN
+F 2 "Connectors_Samtec:SL-105-X-XX_1x05" H 2150 3450 50  0001 C CNN
 F 3 "" H 2150 3450 50  0001 C CNN
 	1    2150 3450
@@
 $EndComp
 $Comp
-L conn:Conn_01x02 P20
+L RCTX-rescue:Conn_01x02-conn P?
 U 1 1 5ED823AF
 P 7550 4950
-F 0 "P20" H 7500 5050 50  0000 L CNN
+AR Path="/5ED823AF" Ref="P?"  Part="1"
+AR Path="/5038E44C/5ED823AF" Ref="P21"  Part="1"
+F 0 "P21" H 7500 5050 50  0000 L CNN
 F 1 "TX_VCC" V 7650 4750 50  0000 L CNN
-F 2 "" H 7550 4950 50  0001 C CNN
+F 2 "Connectors_Samtec:SL-102-X-XX_1x02" H 7550 4950 50  0001 C CNN
 F 3 "~" H 7550 4950 50  0001 C CNN
 	1    7550 4950
@@
 F 0 "U2" H 4850 2600 50  0000 L CNN
 F 1 "MB504L" H 4400 3000 50  0000 L CNN
-F 2 "" H 4550 3000 50  0001 C CNN
+F 2 "Housings_DIP:DIP-8_W7.62mm" H 4550 3000 50  0001 C CNN
 F 3 "" H 4550 3000 50  0001 C CNN
 	1    4550 3000
@@
 $EndComp
 $Comp
-L diode:BAV99 D1
+L RCTX-rescue:BAV99-diode D1
 U 2 1 5D928E22
 P 3800 3000
@@
 $EndComp
 $Comp
-L diode:BAV99 D1
+L RCTX-rescue:BAV99-diode D1
 U 1 1 5D929781
 P 3550 3000
@@
 $EndComp
 $Comp
-L device:L L1
+L RCTX-rescue:L-device L1
 U 1 1 5D92F604
 P 3300 3000
 F 0 "L1" H 3350 2650 50  0000 R CNN
 F 1 "Pickup coil" V 3200 3200 50  0000 R CNN
-F 2 "" H 3300 3000 50  0001 C CNN
+F 2 "Inductors_THT:L_Axial_L5.3mm_D2.2mm_P2.54mm_Vertical_Vishay_IM-1" H 3300 3000 50  0001 C CNN
 F 3 "" H 3300 3000 50  0001 C CNN
 	1    3300 3000
@@
 Connection ~ 3800 3250
 $Comp
-L device:C C2
+L RCTX-rescue:C-device C1
 U 1 1 5D943AA6
 P 4000 3800
-F 0 "C2" H 3885 3754 50  0000 R CNN
+F 0 "C1" H 3885 3754 50  0000 R CNN
 F 1 "100nF" H 3885 3845 50  0000 R CNN
-F 2 "" H 4038 3650 50  0001 C CNN
+F 2 "Capacitors_THT:C_Disc_D3.0mm_W1.6mm_P2.50mm" H 4038 3650 50  0001 C CNN
 F 3 "" H 4000 3800 50  0001 C CNN
 	1    4000 3800
@@
 Connection ~ 4450 2450
 $Comp
-L device:R R2
+L RCTX-rescue:R-device R1
 U 1 1 5D962B9C
 P 5100 3800
-F 0 "R2" H 5170 3846 50  0000 L CNN
+F 0 "R1" H 5170 3846 50  0000 L CNN
 F 1 "2k2" H 5170 3755 50  0000 L CNN
-F 2 "" V 5030 3800 50  0001 C CNN
+F 2 "Resistors_THT:R_Axial_DIN0204_L3.6mm_D1.6mm_P1.90mm_Vertical" V 5030 3800 50  0001 C CNN
 F 3 "" H 5100 3800 50  0001 C CNN
 	1    5100 3800
@@
 	5100 2900 5100 3650
 $Comp
-L device:C C5
+L RCTX-rescue:C-device C4
 U 1 1 5D965D0C
 P 5350 2900
-F 0 "C5" V 5098 2900 50  0000 C CNN
+F 0 "C4" V 5098 2900 50  0000 C CNN
 F 1 "1nF" V 5189 2900 50  0000 C CNN
-F 2 "" H 5388 2750 50  0001 C CNN
+F 2 "Capacitors_THT:C_Disc_D3.0mm_W1.6mm_P2.50mm" H 5388 2750 50  0001 C CNN
 F 3 "" H 5350 2900 50  0001 C CNN
 	1    5350 2900
@@
 Connection ~ 5100 2900
 $Comp
-L transistors:BC547 Q1
+L RCTX-rescue:BC547-transistors Q1
 U 1 1 5D96A0DB
 P 5800 2900
@@
 $EndComp
 $Comp
-L device:R R3
+L RCTX-rescue:R-device R2
 U 1 1 5D96B20F
 P 6500 2950
-F 0 "R3" H 6430 2904 50  0000 R CNN
+F 0 "R2" H 6430 2904 50  0000 R CNN
 F 1 "15k" H 6430 2995 50  0000 R CNN
-F 2 "" V 6430 2950 50  0001 C CNN
+F 2 "Resistors_THT:R_Axial_DIN0204_L3.6mm_D1.6mm_P1.90mm_Vertical" V 6430 2950 50  0001 C CNN
 F 3 "" H 6500 2950 50  0001 C CNN
 	1    6500 2950
@@
 $EndComp
 $Comp
-L device:L L2
+L RCTX-rescue:L-device L2
 U 1 1 5D96B951
 P 6500 3500
 F 0 "L2" H 6456 3454 50  0000 R CNN
 F 1 "10uH" H 6456 3545 50  0000 R CNN
-F 2 "" H 6500 3500 50  0001 C CNN
+F 2 "Inductors_THT:L_Axial_L5.3mm_D2.2mm_P2.54mm_Vertical_Vishay_IM-1" H 6500 3500 50  0001 C CNN
 F 3 "" H 6500 3500 50  0001 C CNN
 	1    6500 3500
@@
 Connection ~ 4650 4050
 $Comp
-L regul:LM78L05_TO92 U1
+L RCTX-rescue:LM78L05_TO92-regul U1
 U 1 1 5D9720E2
 P 4400 4550
@@
 $EndComp
 $Comp
-L device:C C4
+L RCTX-rescue:C-device C3
 U 1 1 5D974D6A
 P 4800 4300
-F 0 "C4" H 4750 4200 50  0000 R CNN
+F 0 "C3" H 4750 4200 50  0000 R CNN
 F 1 "10nF" H 5000 4200 50  0000 R CNN
-F 2 "" H 4838 4150 50  0001 C CNN
+F 2 "Capacitors_THT:C_Disc_D3.0mm_W1.6mm_P2.50mm" H 4838 4150 50  0001 C CNN
 F 3 "" H 4800 4300 50  0001 C CNN
 	1    4800 4300
@@
 $EndComp
 $Comp
-L device:C C3
+L RCTX-rescue:C-device C2
 U 1 1 5D975876
 P 4000 4300
-F 0 "C3" H 3950 4200 50  0000 R CNN
+F 0 "C2" H 3950 4200 50  0000 R CNN
 F 1 "10nF" H 4200 4200 50  0000 R CNN
-F 2 "" H 4038 4150 50  0001 C CNN
+F 2 "Capacitors_THT:C_Disc_D3.0mm_W1.6mm_P2.50mm" H 4038 4150 50  0001 C CNN
 F 3 "" H 4000 4300 50  0001 C CNN
 	1    4000 4300
@@
 PPM_OUT
 $Comp
-L conn:Conn_01x03 P18
+L RCTX-rescue:Conn_01x03-conn P19
 U 1 1 4E4833D2
 P 7550 2050
-F 0 "P18" H 7550 1850 50  0000 C CNN
+F 0 "P19" H 7550 1850 50  0000 C CNN
 F 1 "TX_MOD" V 7650 2050 40  0000 C CNN
-F 2 "" H 7550 2050 50  0001 C CNN
+F 2 "Connectors_Samtec:SL-103-X-XX_1x03" H 7550 2050 50  0001 C CNN
 F 3 "" H 7550 2050 50  0001 C CNN
 	1    7550 2050
@@
 	3200 3250 3200 2650
 $Comp
-L device:Antenna_Shield AE1
+L RCTX-rescue:Antenna_Shield-device AE1
 U 1 1 5DA2F2A1
 P 3200 2450
 F 0 "AE1" H 3120 2489 50  0000 R CNN
 F 1 "Antenna_Shield" H 3120 2398 50  0000 R CNN
-F 2 "" H 3200 2550 50  0001 C CNN
+F 2 "Connectors_Samtec:SL-102-X-XX_1x02" H 3200 2550 50  0001 C CNN
 F 3 "" H 3200 2550 50  0001 C CNN
 	1    3200 2450
@@
 	3150 3200 3150 2800
 $Comp
-L conn:Conn_01x04 P19
+L RCTX-rescue:Conn_01x04-conn P20
 U 1 1 5DE4A168
 P 7550 3950
-F 0 "P19" H 7500 4250 50  0000 L CNN
+F 0 "P20" H 7500 4250 50  0000 L CNN
 F 1 "PWR_BUS" V 7650 3800 50  0000 L CNN
-F 2 "" H 7550 3950 50  0001 C CNN
+F 2 "Connectors_Samtec:SL-104-X-XX_1x04" H 7550 3950 50  0001 C CNN
 F 3 "~" H 7550 3950 50  0001 C CNN
 	1    7550 3950
@@
 NoConn ~ 7350 3950
 $Comp
-L power:+3.3V #PWR?
+L RCTX-rescue:+3.3V-power #PWR07
 U 1 1 5F84CE9B
 P 7050 3750
-F 0 "#PWR?" H 7050 3600 50  0001 C CNN
+F 0 "#PWR07" H 7050 3600 50  0001 C CNN
 F 1 "+3.3V" H 7065 3923 50  0000 C CNN
 F 2 "" H 7050 3750 50  0001 C CNN
@@
 $EndComp
 $Comp
-L power:GND #PWR?
+L RCTX-rescue:GND-power #PWR06
 U 1 1 5F84D89D
 P 5900 4150
-F 0 "#PWR?" H 5900 3900 50  0001 C CNN
+F 0 "#PWR06" H 5900 3900 50  0001 C CNN
 F 1 "GND" H 5905 3977 50  0000 C CNN
 F 2 "" H 5900 4150 50  0001 C CNN
@@
 	5900 4150 5900 4050
 $Comp
-L power:+5V #PWR?
+L RCTX-rescue:+5V-power #PWR05
 U 1 1 5F8530E2
 P 4450 2350
-F 0 "#PWR?" H 4450 2200 50  0001 C CNN
+F 0 "#PWR05" H 4450 2200 50  0001 C CNN
 F 1 "+5V" H 4465 2523 50  0000 C CNN
 F 2 "" H 4450 2350 50  0001 C CNN
