File: kicad/RCTX.kicad_pcb (KiCad board)
At the start: 2 copper layers, 222 parts, among them J1 ROTARY_4, J10 H_RIGHT_JOYSTIC, J11 ROTARY_9, J12 V_RIGHT_JOYSTIC, J13 ROTARY_10, J14 H_LEFT_JOYSTIC, J15 ROTARY_11, J16 V_LEFT_JOYSTIC, J17 ROTARY_12, J18 MULTI_PROP_1, J19 MULTI_PROP_2, J2 ROTARY_5, J20 Conn_01x17, J21 Conn_01x17, J22 Conn_01x17, J23 Conn_01x17, J24 ROTARY_4, J25 ROTARY_5, J26 ROTARY_3, J27 ROTARY_6, J28 ROTARY_2, J29 ROTARY_7, J3 ROTARY_3, J30 ROTARY_1, J31 ROTARY_8, J32 PWR_BUS, J33 H_RIGHT_JOYSTIC, J34 ROTARY_9, J35 V_RIGHT_JOYSTIC, J36 ROTARY_10, J37 H_LEFT_JOYSTIC, J38 ROTARY_11, J39 V_LEFT_JOYSTIC, J4 ROTARY_6, J40 ROTARY_12, J41 MULTI_PROP_1, J42 MULTI_PROP_2, J5 ROTARY_2, J6 ROTARY_7, J7 ROTARY_1, J8 ROTARY_8, J9 PWR_BUS, P1 MULTI_PROP_1, P10 POWER_IN, P11 USB, P12 BUZZ, P13 SW, P14 LEDS, P15 KEYPAD, P16 MULTI_DIGITAL_1, P17 MULTI_DIGITAL_2, P18 RF MODULE, P19 TX_MOD, P2 MULTI_PROP_2, P20 PWR_BUS, P21 TX_VCC, P22 SW, P23 PWR_BUS, P24 TX_VCC, P25 MULTI_DIGITAL_1, P26 PWR_BUS, P27 LEDS, P28 PWR_BUS, P29 MULTI_DIGITAL_2, P3 SD_CARD, P30 PWR_BUS, P31 PWR_BUS, P32 LEDs, P33 DISPLAY, P34 CONN_8, P35 CONN_8, P36 Nokia 5110 Display, P37 CONN_8, P38 CONN_8, P39 KEYBOARD, P4 LEDs, P5 DISPLAY, P6 EJTAG + IO_PORT, P7 TX_MOD, P8 AUX_DB15_PORT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

Commit message: WIP
Parts:
- moved C12 234.3 mm to (233.7, 308.6)
- moved R4 232.6 mm to (237.5, 315.0)
- moved U5 232.0 mm to (232.2, 330.0)
- moved J9 232.0 mm to (194.3, 321.6)
- moved R3 232.0 mm to (253.6, 312.3)
- moved C8 223.6 mm to (325.1, 292.1), turned to 180 degrees
- moved J15 221.7 mm to (189.2, 274.3), turned to 180 degrees
- moved C7 221.7 mm to (221.0, 306.1)
- moved C6 221.3 mm to (285.8, 292.1), turned to 180 degrees
- moved C10 214.4 mm to (242.6, 285.8)
- moved J3 210.9 mm to (334.0, 275.6)
- moved C9 206.8 mm to (283.2, 285.8)
- moved U3 206.6 mm to (320.0, 264.2)
- moved J4 205.6 mm to (334.0, 269.2)
- moved C5 205.1 mm to (322.6, 285.8)
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