File: kicad/VHF_Transceiver.sch (KiCad schematic (older format))
At the start: 47 parts

Commit message: New rx-tx bidirectional amplifier
Parts:
- removed C? (x13): .1, symbol device:C
- removed Q? (x2): 2N3904, TO_SOT_Packages_THT:TO-92_Molded_Narrow, symbol transistors:2N3904
- removed Q? (x2): 2N3906, TO_SOT_Packages_THT:TO-92_Molded_Narrow, symbol transistors:2N3906
- removed R? (x3): 1k, symbol device:R
- removed R? (x6): 680, symbol device:R
- removed R? (x4): 100, symbol device:R
- removed SW?: SW_SPDT, symbol switches:SW_SPDT
Connections:
- wire segments 155 -> 74
