File: kicad/RCTX_ERF32FG12.sch (KiCad schematic (older format))
At the start: 45 parts, among them P1 MULTI_PROP_1, P10 POWER_IN, P12 BUZZ, P14 LEDS, P15 SWITCHES, P2 MULTI_PROP_2, P6 EJTAG + IO_PORT, P8 AUX_DB15_PORT, P9 PWR_BUS

Commit message: Using ERF32FG12 SoC instead of PIC32MX
Parts:
- removed C?: 1u, symbol device:C
- removed C?: 100n, symbol device:C
- removed C?: 4u7, symbol device:C
- removed J? (x2): SPI, symbol conn:Conn_01x03
- removed J? (x2): SPI_USERS, symbol conn:Conn_01x06
- removed J?: BUZZ, symbol conn:Conn_01x01
- removed L?: 4u7, symbol device:L
- removed P1, P?: MULTI_PROP_1, Connectors_Samtec:SL-108-X-XX_1x08, symbol RCTX-rescue:Conn_01x08-conn
- removed P10: POWER_IN, Connectors_Samtec:SL-104-X-XX_1x04, symbol RCTX-rescue:Conn_01x04-conn
- removed P12: BUZZ, Connectors_Samtec:SL-102-X-XX_1x02, symbol RCTX-rescue:Conn_01x02-conn
- removed P14, P?: LEDS, Connectors_Samtec:SL-104-X-XX_1x04, symbol RCTX-rescue:Conn_01x04-conn
- removed P15, P?: SWITCHES, Connectors_Samtec:SL-108-X-XX_1x08, symbol RCTX-rescue:Conn_01x08-conn
- removed P2, P?: MULTI_PROP_2, Connectors_Samtec:SL-108-X-XX_1x08, symbol RCTX-rescue:Conn_01x08-conn
- removed P6: EJTAG + IO_PORT, Connectors_Samtec:SL-108-X-XX_1x08, symbol RCTX-rescue:Conn_01x08-conn
- removed P8: AUX_DB15_PORT, Connectors_Samtec:SL-112-X-XX_1x12, symbol RCTX-rescue:Conn_01x12-conn
- removed P9: PWR_BUS, Connectors_Samtec:SL-104-X-XX_1x04, symbol RCTX-rescue:Conn_01x04-conn
- removed P?: SD_CARD, Connectors_Samtec:SL-104-X-XX_1x04, symbol RCTX-rescue:Conn_01x04-conn
- removed P?: LEDs, Connectors_Samtec:SL-104-X-XX_1x04, symbol RCTX-rescue:Conn_01x04-conn
- removed P?: DISPLAY, Connectors_Samtec:SL-106-X-XX_1x06, symbol RCTX-rescue:Conn_01x05-conn
- removed P? (x2): SW, Connectors_Samtec:SL-102-X-XX_1x02, symbol RCTX-rescue:Conn_01x02-conn
- removed P? (x2): KEYPAD, symbol conn:Conn_01x02
- removed RV1: POT, Potentiometers:Potentiometer_Trimmer_ACP_CA6v_Horizontal, symbol RCTX-rescue:POT_TRIM-device
- removed ZD1: ZENER, Diodes_THT:D_5W_P5.08mm_Vertical_KathodeUp, symbol RCTX-rescue:D_Zener-device
- added C? (x10): 100n, symbol device:C
- added C?: 10u 16V, symbol device:CP
- added C?: 4u7, symbol device:C
- added C? (x11): 1u, symbol device:C
- added C? (x6): 100p, symbol device:C
- added D? (x2): GREEN, symbol device:LED
- added D?: D, symbol device:D
- added D?: RED, symbol device:LED
- added F?: Polyfuse, symbol device:Polyfuse
- added J?: USB_OTG, symbol conn:USB_OTG
- added J?: 50 Ohm Antenna, symbol conn:Conn_Coaxial
- added L?: 4u7, symbol device:L
- added L? (x6): L, symbol device:L
- added P?: ARM 20 Pin Header, symbol conn:Conn_02x10_Odd_Even
- added P?: POWER_IN, Connectors_Samtec:SL-104-X-XX_1x04, symbol RCTX-rescue:Conn_01x04-conn
- added P? (x2): KEYPAD, symbol conn:Conn_02x03_Odd_Even
- added P?: SWITCHES, symbol conn:Conn_02x08_Odd_Even
- added P?: SW, symbol conn:Conn_02x02_Odd_Even
- added P?: BUZZ, symbol conn:Conn_02x01
- added P?: POWER, symbol conn:Conn_02x03_Odd_Even
- added P?: SD Card, symbol conn:Conn_02x05_Odd_Even
- added P?: Nokia 5110 display, symbol conn:Conn_02x06_Odd_Even
- added P?: Left SW LEDs, symbol conn:Conn_02x08_Odd_Even
- added P?: Right SW LEDs, symbol conn:Conn_02x07_Odd_Even
- added P?: MULTI_PROP_1, symbol conn:Conn_02x10_Odd_Even
- added P?: MULTI_PROP_2, symbol conn:Conn_02x10_Odd_Even
- added P?: AUX_DB15_PORT, symbol conn:Conn_02x15_Counter_Clockwise
- added R? (x3): 1k, symbol device:R
- added RV?: POT, Potentiometers:Potentiometer_Trimmer_ACP_CA6v_Horizontal, symbol RCTX-rescue:POT_TRIM-device
- added U?: FT232RL, Housings_SSOP:SSOP-28_5.3x10.2mm_Pitch0.65mm, symbol ftdi:FT232RL
- added U?: LM1117-5.0, symbol regul:LM1117-5.0
- added U?: KTD2061, symbol Kinetic:KTD2061
- added U?: SC18IS602B, symbol nxp_sc18is602b:SC18IS602B
- added U? (x2): MAX2650, smd-semi:SOT-143, symbol maxim_1:MAX2650
- added U?: ADE-1+, RF_Mini-Circuits:Mini-Circuits_CD542_LandPatternPL-052, symbol RF_Mixer:ADE-1+
- added U? (x2): TLV70245_SOT23-5, TO_SOT_Packages_SMD:SOT-23-5, symbol regul:TLV70245_SOT23-5
- added Y?: Si500DFAD100M000 / Si511NCB100M000C, Si500D, symbol Si500D:Si500D
- added ZD?: ZENER, Diodes_THT:D_5W_P5.08mm_Vertical_KathodeUp, symbol RCTX-rescue:D_Zener-device
Connections:
- net labels added: INTn, MASTER|SLAVEn, PPM_IN, PPM_OUT, RESETn, RF_ENABLE, RF_RX_EN, RF_RX_VCC, RF_TX_EN, RF_TX_VCC, SCL, SDA, SWDCLK-TMS, SWDIO-TCK, SWDO-TDO, TDI, UART_CTS, UART_RTS, UART_RX, UART_TX, USB_RX, USB_TX, VBATT
- net labels removed: +BATT, LED1, LED2, LED3, LED4
- wire segments 160 -> 661
- no-connect marks 0 -> 12
Other:
- note added: "I/O connectors"
- note added: "I2C driver for status LEDs"
- note added: "I2C to SPI bridge for SD Card and Nokia 5110 display"
- note added: "Low pass filter fc: 80 MHz"
- note added: "MCU"
- note added: "Main power source and USB interface"
- note added: "RX and TX frontend power"
- note added: "VCC"
- note removed: "+3.3V"
- note removed: "+5V"
- note removed: "/PWM"
- note removed: "CLK"
- note removed: "CTS1"
- note removed: "CTS2"
- note removed: "DIN"
- note removed: "LCD /CE"
- note removed: "LCD /RESET"
- note removed: "LE"
- note removed: "LEDS /PWM"
- note removed: "LEDs CLK"
- note removed: "LEDs LE"
- note removed: "PPM_IN"
- note removed: "PPM_OUT"
- note removed: "Pins cfg:\n\nAIN + ADC"
- note removed: "Pins cfg:\n\nDIN + PULL_UP"
- note removed: "Pins cfg:\n\nDIN\n"
- note removed: "Pins cfg:\n\nDOUT"
- note removed: "Pins cfg:\n\nDOUT + WAVE_GEN"
- note removed: "RTS1"
- note removed: "RTS2"
- note removed: "RX1"
- note removed: "RX2"
- note removed: "SCL"
- note removed: "SDA"
- note removed: "SS/CS"
- note removed: "TCK"
- note removed: "TDI"
- note removed: "TDO"
- note removed: "TMS"
- note removed: "TX1"
- note removed: "TX2"
- note removed: "nSRST"
- moved on the sheet: C?, L?, R?, SW?, U?, Y?
