File: kicad/DisplayI2C.sch (KiCad schematic (older format))
At the start: 41 parts

Commit message: Splitting leds in dispay schema
Parts:
- removed D? (x36): LED, symbol device:LED
- removed J?: Conn_01x04, symbol conn:Conn_01x04
- added D? (x36): LED, symbol device:LED
- added J? (x2): Right Switches LED Display, symbol conn:Conn_01x07
- added J? (x2): Status LEDs, symbol conn:Conn_01x03
- added J? (x2): Left Switches LED Display, symbol conn:Conn_01x08
Connections:
- net labels added: +3.3V, +3v3, LEDA1, LEDA2, LEDA3, LEDA4, LEDB1, LEDB2, LEDB3, LEDB4, LEDC1, LEDC2, LEDC3, LEDC4, SCL, SDA
- wire segments 207 -> 261
Other:
- note added: "Left Switches LED display"
- note added: "Right Switches LED display"
- note added: "Status LEDs"
- moved on the sheet: C?, R?, U?

Commit message: Using ERF32FG12 SoC instead of PIC32MX
Parts:
- removed C?: 10u 16V, symbol device:C
- removed J? (x2): Right Switches LED Display, symbol conn:Conn_01x07
- removed J? (x2): Status LEDs, symbol conn:Conn_01x03
- removed J? (x2): Left Switches LED Display, symbol conn:Conn_01x08
- removed R? (x2): 10k, symbol device:R
- removed U?: KTD2061, symbol Kinetic:KTD2061
- added P?: Right Switches LED Display, symbol conn:Conn_02x07_Odd_Even
- added P?: Left Switches LED Display, symbol conn:Conn_02x08_Odd_Even
- added P?: Status LEDs, symbol conn:Conn_02x03_Odd_Even
Connections:
- net labels removed: +3.3V, +3v3, SCL, SDA
- wire segments 261 -> 201
Other:
- moved on the sheet: D?
