File: kicad/RCRX_ERF32MG12.sch (KiCad schematic (older format))
At the start: 98 parts

Commit message: Replacing discrete components rf filters with Mini-Circuits single chip filters
Parts:
- removed C? (x2): 5.1p, symbol device:C
- removed C?: 33p, symbol device:C
- removed L? (x2): 22n, symbol device:L
- removed U?: JSW2-63DR+, symbol RF_Mixer:JSW2-63DR+
- added C?: 43p, symbol device:C
- added C? (x2): 2.2p, symbol device:C
- added C?: 1p, symbol device:C
- added L? (x2): 3n, symbol device:L
- added L? (x2): 62n, symbol device:L
- added L?: 130n, symbol device:L
- added L?: 82n, symbol device:L
- C?: value 11p -> 43p
- C?: value 75p -> 56p
- C?: value 33p -> 56p
- C? (x2): value 75p -> 68p
- L?: value 150n -> 82n
- L?: value 150n -> 180n
Connections:
- wire segments 446 -> 445
Other:
- note added: "High Band harmonics suppressor\n5th order Chebyshev band pass filter fc: 400-500 MHz"
- note removed: "High Band harmonics suppressor\n5th order Chebyshev low\npass filter fc: 460 MHz"
- moved on the sheet: C?, J?, L?
