File: kicad/RCRX_ERF32MG12.kicad_sch (KiCad schematic)
At the start: 96 parts, among them J20 USB_OTG, J21 USB, J22 USB, J5 Micro_SD_Card, P10 LEDs, P9 BUZZ, SW1 RESET, U1 MAX2650, U11 USB6B1, U12 MAX2650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

Commit message: Added HEX rotary encoder and DIP switch for RX SUB ID selection in the receiver circuit. Updated README.md
Parts:
- removed P?: POWER_IN, Connectors_Samtec:SL-104-X-XX_1x04, symbol RCTX-rescue:Conn_01x04-conn
- removed RV?: POT, Potentiometers:Potentiometer_Trimmer_ACP_CA6v_Horizontal, symbol RCTX-rescue:POT_TRIM-device
- removed ZD?: ZENER, Diodes_THT:D_5W_P5.08mm_Vertical_KathodeUp, symbol RCTX-rescue:D_Zener-device
- added D? (x12): 1N4148, Diodes_THT:D_5W_P5.08mm_Vertical_KathodeUp, symbol RCTX-rescue:D-device
- added HEX_SW1: RX_SUB_ID, symbol switches:SW_Coded
- added J8: POWER, symbol Connector_Generic:Conn_01x02
- added SW2: RX_SUB_ID_EN, symbol Switch:SW_DIP_x01
- HEX_SW?: value MODEL_ID -> RX_ID
Connections:
- net +BATT: now also J8.1 (Pin_1)
- net GND: now also J8.2 (Pin_2)
- net I2C_SCL: now also U?.33 (PB13); no longer U?.32 (PB12)
- net I2C_SDA: now also U?.32 (PB12); no longer U?.31 (PB11)
- net at U?.24 (PD15): now also SW2.2
- new net: D?.1 (K), D?.1 (K), D?.1 (K), U?.27 (PA2)
- new net: D?.1 (K), D?.1 (K), D?.1 (K), U?.28 (PA3)
- new net: D?.1 (K), D?.1 (K), D?.1 (K), U?.29 (PA4)
- new net: D?.1 (K), D?.1 (K), D?.1 (K), U?.30 (PA5)
- new net: HEX_SW1.1 (CM), SW2.1, U?.31 (PB11)
- new net: D?.2 (A), HEX_SW?.2 (D0) (x2)
- new net: D?.2 (A), HEX_SW?.3 (D1) (x2)
- new net: D?.2 (A), HEX_SW?.4 (D2) (x2)
- new net: D?.2 (A), HEX_SW?.5 (D3) (x2)
- new net: D?.2 (A), HEX_SW1.2 (D0)
- new net: D?.2 (A), HEX_SW1.3 (D1)
- new net: D?.2 (A), HEX_SW1.5 (D3)
- new net: D?.2 (A), HEX_SW1.4 (D2)
- no-connect marks 13 -> 11
Other:
- note removed: "AMPEROMETER"
- moved on the sheet: C1, C18, C2, C20, C21, C22, C?, HEX_SW?, J?, L?, P?, R?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

Commit message: Update README.md Updated the Decoder description
Parts:
- removed D? (x4): 1N4148, Diodes_THT:D_5W_P5.08mm_Vertical_KathodeUp, symbol RCTX-rescue:D-device
- removed HEX_SW?: RF_BAND_SEL, symbol switches:SW_Coded
- removed P?: I2C_BUS, symbol conn:Conn_01x04
- added D? (x4): 1N4148, Diodes_THT:D_5W_P5.08mm_Vertical_KathodeUp, symbol RCTX-rescue:D-device
- added HEX_SW2: RX_BAND_SEL, symbol switches:SW_Coded
- added P4: I2C_BUS, symbol conn:Conn_01x04
- added P5: DSC_BUS, symbol conn:Conn_01x04
- HEX_SW1: value RX_SUB_ID -> RX_ID
- HEX_SW?: value RX_ID -> RX_SUB_ID
- SW2: value RX_SUB_ID_EN -> RX_RADIO_EN
Connections:
- net +5V: now also P4.3 (Pin_3)
- net +BATT: now also P5.3 (Pin_3)
- net CRSF_RX: now also P?.1 (Pin_1); no longer P?.2 (Pin_2)
- net CRSF_TX: now also P?.2 (Pin_2); no longer P?.1 (Pin_1)
- net GND: now also P4.4 (Pin_4), P5.4 (Pin_4)
- net I2C_SCL: now also P4.1 (Pin_1)
- net I2C_SDA: now also P4.2 (Pin_2)
- net at SW2.2, U?.24 (PD15): now also HEX_SW2.1 (CM)
- net at U?.25 (PA0): now also HEX_SW1.1 (CM)
- net at D?.1 (K), D?.1 (K), U?.27 (PA2): now also D?.1 (K)
- net at D?.1 (K), D?.1 (K), U?.28 (PA3): now also D?.1 (K)
- net at D?.1 (K), D?.1 (K), U?.29 (PA4): now also D?.1 (K)
- net at D?.1 (K), D?.1 (K), U?.30 (PA5): now also D?.1 (K)
- net at SW2.1, U?.31 (PB11): no longer HEX_SW1.1 (CM)
- net SIGNAL: now reaches U?.47 (PC10)
- net SIGNAL: now also P5.2 (Pin_2)
- net TELEMETRY: now reaches U?.48 (PC11)
- net TELEMETRY: now also P5.1 (Pin_1)
- new net: D?.2 (A), HEX_SW2.3 (D1)
- new net: D?.2 (A), HEX_SW2.5 (D3)
- new net: D?.2 (A), HEX_SW2.4 (D2)
- new net: D?.2 (A), HEX_SW2.2 (D0)
- no-connect marks 11 -> 9
Other:
- moved on the sheet: D?, HEX_SW1, HEX_SW?, P?, SW2
